File: Hardware/rf-receiver.sch (KiCad schematic (older format))
At the start: 28 parts, among them IC1 ATSAMD21G18A-AU, P1 ROT_ENC, P2 USB_B, SW1 BTN1, SW2 BTN2, SW3 BTN3, U5 74HC14, Y1 Crystal_Small

Commit message: Second actual HW commit
First finished draft of HW layout and PCB design.
Parts:
- removed P2: USB_B, Connect:USB_B, symbol Connector:USB_B
- removed R3, R4: 10kohm, Resistors_SMD:R_0805_HandSoldering, symbol Device:R_Small
- added MH1, MH2, MH3, MH4: MountingHole_Pad, MountingHole:MountingHole_4.3mm_M4_Pad, symbol Mechanical:MountingHole_Pad
- C1: renamed from C11; footprint Capacitors_SMD:C_0805_HandSoldering -> Capacitor_SMD:C_0402_1005Metric
- C2: renamed from C12; footprint Capacitors_SMD:C_0805_HandSoldering -> Capacitor_SMD:C_0402_1005Metric
- C3: renamed from C9; footprint Capacitors_SMD:C_0805_HandSoldering -> Capacitor_SMD:C_0402_1005Metric
- C4: renamed from C10; footprint Capacitors_SMD:C_0805_HandSoldering -> Capacitor_SMD:C_0402_1005Metric
- C5: renamed from C13; footprint Capacitors_SMD:C_0805_HandSoldering -> Capacitor_SMD:C_0402_1005Metric
- C6: renamed from C14; footprint Capacitors_SMD:C_0805_HandSoldering -> Capacitor_SMD:C_0402_1005Metric
- C7: renamed from C15; footprint Capacitors_SMD:C_0805_HandSoldering -> Capacitor_SMD:C_0402_1005Metric
- C8: renamed from C16; footprint Capacitors_SMD:C_0805_HandSoldering -> Capacitor_SMD:C_0402_1005Metric
- IC1: footprint ATSAMD21G18A-AU:QFP50P900X900X120-48N -> Package_QFP:TQFP-48_7x7mm_P0.5mm
- P1: footprint Pin_Headers:Pin_Header_Straight_1x03_Pitch2.00mm -> Connector_PinHeader_2.54mm:PinHeader_1x03_P2.54mm_Vertical
- R1, R10, R2, R5, R6, R7, R8, R9: footprint Resistors_SMD:R_0805_HandSoldering -> Resistor_SMD:R_0402_1005Metric
- SW1, SW2, SW3: footprint Pin_Headers:Pin_Header_Straight_1x02_Pitch2.54mm -> Connector_PinHeader_2.54mm:PinHeader_1x02_P2.54mm_Vertical
- U1: renamed from U5; footprint Housings_SSOP:TSSOP-14_4.4x5mm_Pitch0.65mm -> Package_SO:TSSOP-14_4.4x5mm_P0.65mm
- W1: renamed from W3; footprint Wire_Pads:SolderWirePad_single_2mmDrill -> TestPoint:TestPoint_THTPad_2.0x2.0mm_Drill1.0mm
- W2: renamed from W4; footprint Wire_Pads:SolderWirePad_single_2mmDrill -> TestPoint:TestPoint_THTPad_2.0x2.0mm_Drill1.0mm
- Y1: footprint Crystals:Crystal_SMD_G8-2pin_3.2x1.5mm_HandSoldering -> Crystal:Crystal_SMD_3215-2Pin_3.2x1.5mm
Connections:
- wire segments 162 -> 159

Commit message: Added BOM
Added BOM.csv
Added Micro-USB
Parts:
- added J3: USB_B_Micro, Connector_USB:USB_Micro-B_Molex-105017-0001, symbol Connector:USB_B_Micro
- added R3, R4: R_Small, Resistor_SMD:R_0402_1005Metric, symbol Device:R_Small
- MH1, MH2, MH3, MH4: footprint MountingHole:MountingHole_4.3mm_M4_Pad -> MountingHole:MountingHole_2.7mm_M2.5_Pad
Connections:
- net labels added: USB_D+, USB_D-, USB_VCC
- net labels removed: USB/DM, USB/DP, USB/VCC
- wire segments 159 -> 171
- no-connect marks 10 -> 11
Changed lines of the file:
@@
 EESchema Schematic File Version 4
+LIBS:rf-receiver-cache
 EELAYER 26 0
 EELAYER END
@@
 Connection ~ 4200 1500
 Text Label 3890 3850 0    60   ~ 0
-USB/DM
+USB_D-
 Text Label 3890 3950 0    60   ~ 0
-USB/DP
+USB_D+
 NoConn ~ 4400 3650
-Wire Wire Line
-	4400 3750 3890 3750
-Text Label 3890 3750 0    60   ~ 0
-USB/VCC
 NoConn ~ 1200 1300
 NoConn ~ 1200 1400
@@
 F 0 "MH1" H 1250 5751 50  0000 L CNN
 F 1 "MountingHole_Pad" H 1250 5660 50  0000 L CNN
-F 2 "MountingHole:MountingHole_4.3mm_M4_Pad" H 1150 5700 50  0001 C CNN
+F 2 "MountingHole:MountingHole_2.7mm_M2.5_Pad" H 1150 5700 50  0001 C CNN
 F 3 "~" H 1150 5700 50  0001 C CNN
 	1    1150 5700
@@
 F 0 "MH2" H 1475 5751 50  0000 L CNN
 F 1 "MountingHole_Pad" H 1475 5660 50  0000 L CNN
-F 2 "MountingHole:MountingHole_4.3mm_M4_Pad" H 1375 5700 50  0001 C CNN
+F 2 "MountingHole:MountingHole_2.7mm_M2.5_Pad" H 1375 5700 50  0001 C CNN
 F 3 "~" H 1375 5700 50  0001 C CNN
 	1    1375 5700
@@
 F 0 "MH3" H 1700 5751 50  0000 L CNN
 F 1 "MountingHole_Pad" H 1700 5660 50  0000 L CNN
-F 2 "MountingHole:MountingHole_4.3mm_M4_Pad" H 1600 5700 50  0001 C CNN
+F 2 "MountingHole:MountingHole_2.7mm_M2.5_Pad" H 1600 5700 50  0001 C CNN
 F 3 "~" H 1600 5700 50  0001 C CNN
 	1    1600 5700
@@
 F 0 "MH4" H 1900 5751 50  0000 L CNN
 F 1 "MountingHole_Pad" H 1900 5660 50  0000 L CNN
-F 2 "MountingHole:MountingHole_4.3mm_M4_Pad" H 1800 5700 50  0001 C CNN
+F 2 "MountingHole:MountingHole_2.7mm_M2.5_Pad" H 1800 5700 50  0001 C CNN
 F 3 "~" H 1800 5700 50  0001 C CNN
 	1    1800 5700
@@
 	1800 5875 1800 5800
 Connection ~ 1600 5875
+$Comp
+L Connector:USB_B_Micro J3
+U 1 1 5C49A3F1
+P 1275 7075
+F 0 "J3" H 1330 7542 50  0000 C CNN
+F 1 "USB_B_Micro" H 1330 7451 50  0000 C CNN
+F 2 "Connector_USB:USB_Micro-B_Molex-105017-0001" H 1425 7025 50  0001 C CNN
+F 3 "~" H 1425 7025 50  0001 C CNN
+	1    1275 7075
+	1    0    0    -1
+$EndComp
+$Comp
+L Device:R_Small R4
+U 1 1 5C49A683
+P 2125 7050
+F 0 "R4" H 2184 7096 50  0000 L CNN
+F 1 "R_Small" H 2184 7005 50  0000 L CNN
+F 2 "Resistor_SMD:R_0402_1005Metric" H 2125 7050 50  0001 C CNN
+F 3 "~" H 2125 7050 50  0001 C CNN
+	1    2125 7050
+	1    0    0    -1
+$EndComp
+$Comp
+L Device:R_Small R3
+U 1 1 5C49A709
+P 1900 6875
+F 0 "R3" V 1704 6875 50  0000 C CNN
+F 1 "R_Small" V 1795 6875 50  0000 C CNN
+F 2 "Resistor_SMD:R_0402_1005Metric" H 1900 6875 50  0001 C CNN
+F 3 "~" H 1900 6875 50  0001 C CNN
+	1    1900 6875
+	0    1    1    0
+$EndComp
+Wire Wire Line
+	1800 6875 1575 6875
+Wire Wire Line
+	2000 6875 2125 6875
+Wire Wire Line
+	2125 6875 2125 6950
+$Comp
+L power:GND #PWR0108
+U 1 1 5C4AA3F5
+P 2125 7525
+F 0 "#PWR0108" H 2125 7275 50  0001 C CNN
+F 1 "GND" H 2130 7352 50  0000 C CNN
+F 2 "" H 2125 7525 50  0001 C CNN
+F 3 "" H 2125 7525 50  0001 C CNN
+	1    2125 7525
+	1    0    0    -1
+$EndComp
+Wire Wire Line
+	2125 7525 2125 7500
+Wire Wire Line
+	1275 7475 1275 7500
+Wire Wire Line
+	1275 7500 2125 7500
+Connection ~ 2125 7500
+Wire Wire Line
+	2125 7500 2125 7150
+Wire Wire Line
+	1275 7500 1175 7500
+Wire Wire Line
+	1175 7500 1175 7475
+Connection ~ 1275 7500
+NoConn ~ 1575 7275
+Wire Wire Line
+	1985 7075 1575 7075
+Wire Wire Line
+	1575 7175 1985 7175
+Text Label 1985 7175 2    60   ~ 0
+USB_D-
+Text Label 1985 7075 2    60   ~ 0
+USB_D+
+Text Label 3900 3750 0    60   ~ 0
+USB_VCC
+Wire Wire Line
+	4400 3750 3900 3750
+Text Label 2200 6875 0    60   ~ 0
+USB_VCC
+Wire Wire Line
+	2125 6875 2200 6875
+Connection ~ 2125 6875
 $EndSCHEMATC

Commit message: HW PCB changes
Added IBOM
Added extra spacing between 0402 components.
Parts:
- C1: footprint Capacitor_SMD:C_0402_1005Metric -> Resistor_SMD:R_1206_3216Metric
Changed lines of the file:
@@
 F 0 "C1" H 3810 1370 50  0000 L CNN
 F 1 "15pF" H 3700 1200 50  0000 L CNN
-F 2 "Capacitor_SMD:C_0402_1005Metric" H 3800 1300 50  0001 C CNN
+F 2 "Resistor_SMD:R_1206_3216Metric" H 3800 1300 50  0001 C CNN
 F 3 "" H 3800 1300 50  0000 C CNN
 	1    3800 1300

Commit message: HW rev1
Parts:
- removed J3: USB_B_Micro, Connector_USB:USB_Micro-B_Molex-105017-0001, symbol Connector:USB_B_Micro
- added C55: C_Small, Capacitor_SMD:C_0603_1608Metric, symbol Device:C_Small
- added J3: USB_C_Receptacle, athir:DX07S024JJ, symbol Connector:USB_C_Receptacle
- C1: footprint Resistor_SMD:R_1206_3216Metric -> Capacitor_SMD:C_0603_1608Metric
- C2, C3, C4, C5, C6, C7, C8: footprint Capacitor_SMD:C_0402_1005Metric -> Capacitor_SMD:C_0603_1608Metric
- R1, R10, R2, R3, R4, R5, R6, R7, R8, R9: footprint Resistor_SMD:R_0402_1005Metric -> Resistor_SMD:R_0603_1608Metric
Connections:
- wire segments 171 -> 189
- no-connect marks 11 -> 22
