File: Hardware/AD9954sheet.sch (KiCad schematic (older format))
At the start: 39 parts, among them IC2 AD9954

Commit message: Second actual HW commit
First finished draft of HW layout and PCB design.
Parts:
- added C54: 100nF, Capacitor_SMD:C_0402_1005Metric, symbol Device:C_Small
- C17: renamed from C23; footprint Capacitors_SMD:C_0805_HandSoldering -> Capacitor_SMD:C_0402_1005Metric
- C18: renamed from C24; footprint Capacitors_SMD:C_0805_HandSoldering -> Capacitor_SMD:C_0402_1005Metric
- C19: renamed from C25; footprint Capacitors_SMD:C_0805_HandSoldering -> Capacitor_SMD:C_0402_1005Metric
- C20: renamed from C26; footprint Capacitors_SMD:C_0805_HandSoldering -> Capacitor_SMD:C_0402_1005Metric
- C21: renamed from C27; footprint Capacitors_SMD:C_0805_HandSoldering -> Capacitor_SMD:C_0402_1005Metric
- C22: renamed from C29; footprint Capacitors_SMD:C_0805_HandSoldering -> Capacitor_SMD:C_0402_1005Metric
- C23: renamed from C30; footprint Capacitors_SMD:C_0805_HandSoldering -> Capacitor_SMD:C_0402_1005Metric
- C24: renamed from C32; footprint Capacitors_SMD:C_0805_HandSoldering -> Capacitor_SMD:C_0402_1005Metric
- C25: renamed from C34; footprint Capacitors_SMD:C_0805_HandSoldering -> Capacitor_SMD:C_0402_1005Metric
- C26: renamed from C36; footprint Capacitors_SMD:C_0805_HandSoldering -> Capacitor_SMD:C_0402_1005Metric
- C27: renamed from C38; footprint Capacitors_SMD:C_0805_HandSoldering -> Capacitor_SMD:C_0402_1005Metric
- C28: renamed from C40; footprint Capacitors_SMD:C_0805_HandSoldering -> Capacitor_SMD:C_0402_1005Metric
- C29: renamed from C41; footprint Capacitors_SMD:C_0805_HandSoldering -> Capacitor_SMD:C_0402_1005Metric
- C30: renamed from C43; footprint Capacitors_SMD:C_0805_HandSoldering -> Capacitor_SMD:C_0402_1005Metric
- C31: renamed from C44; footprint Capacitors_SMD:C_0805_HandSoldering -> Capacitor_SMD:C_0402_1005Metric
- C32: renamed from C45; footprint Capacitors_SMD:C_0805_HandSoldering -> Capacitor_SMD:C_0402_1005Metric
- C33: renamed from C46; footprint Capacitors_SMD:C_0805_HandSoldering -> Capacitor_SMD:C_0402_1005Metric
- C34: renamed from C47; footprint Capacitors_SMD:C_0805_HandSoldering -> Capacitor_SMD:C_0402_1005Metric
- C35: renamed from C48; footprint Capacitors_SMD:C_0805_HandSoldering -> Capacitor_SMD:C_0402_1005Metric
- C36: renamed from C49; footprint Capacitors_SMD:C_0805_HandSoldering -> Capacitor_SMD:C_0402_1005Metric
- C37: renamed from C50; footprint Capacitors_SMD:C_0805_HandSoldering -> Capacitor_SMD:C_0402_1005Metric
- C38: renamed from C51; footprint Capacitors_SMD:C_0805_HandSoldering -> Capacitor_SMD:C_0402_1005Metric
- C39: renamed from C52; footprint Capacitors_SMD:C_0805_HandSoldering -> Capacitor_SMD:C_0402_1005Metric
- C40: renamed from C53; footprint Capacitors_SMD:C_0805_HandSoldering -> Capacitor_SMD:C_0402_1005Metric
- C41: renamed from C54; footprint Capacitors_SMD:C_0805_HandSoldering -> Capacitor_SMD:C_0402_1005Metric
- C42: renamed from C55; footprint Capacitors_SMD:C_0805_HandSoldering -> Capacitor_SMD:C_0402_1005Metric
- IC2: footprint Housings_QFP:TQFP-48-1EP_7x7mm_Pitch0.5mm -> Package_QFP:TQFP-48-1EP_7x7mm_P0.5mm_EP3.5x3.5mm
- L2: renamed from L5; footprint Capacitors_SMD:C_0805_HandSoldering -> Inductor_SMD:L_0402_1005Metric
- L3: renamed from L6; footprint Capacitors_SMD:C_0805_HandSoldering -> Inductor_SMD:L_0402_1005Metric
- L4: renamed from L7; footprint Capacitors_SMD:C_0805_HandSoldering -> Inductor_SMD:L_0402_1005Metric
- L5: renamed from L8; footprint Capacitors_SMD:C_0805_HandSoldering -> Inductor_SMD:L_0402_1005Metric
- L6: renamed from L9; footprint Capacitors_SMD:C_0805_HandSoldering -> Inductor_SMD:L_0402_1005Metric
- L7: renamed from L10; footprint Capacitors_SMD:C_0805_HandSoldering -> Inductor_SMD:L_0402_1005Metric
- R13: footprint Resistors_SMD:R_0805_HandSoldering -> Resistor_SMD:R_0402_1005Metric
- R14, R15: value 25ohm -> 50ohm; footprint Resistors_SMD:R_0805_HandSoldering -> Resistor_SMD:R_0402_1005Metric
- R16: renamed from R18; footprint Resistors_SMD:R_0805_HandSoldering -> Resistor_SMD:R_0402_1005Metric
- R17: renamed from R19; footprint Resistors_SMD:R_0805_HandSoldering -> Resistor_SMD:R_0402_1005Metric
- XTAL1: footprint Crystals:Crystal_SMD_3225-4pin_3.2x2.5mm_HandSoldering -> Crystal:Crystal_SMD_3225-4Pin_3.2x2.5mm_HandSoldering
Connections:
- wire segments 173 -> 183

Commit message: HW PCB changes
Added IBOM
Added extra spacing between 0402 components.
Parts:
- R14, R15, R17: footprint Resistor_SMD:R_0402_1005Metric -> Resistor_SMD:R_0603_1608Metric
Changed lines of the file:
@@
 F 0 "R17" H 6580 3220 50  0000 L CNN
 F 1 "50ohm" H 6250 3200 50  0000 L CNN
-F 2 "Resistor_SMD:R_0402_1005Metric" H 6550 3200 50  0001 C CNN
+F 2 "Resistor_SMD:R_0603_1608Metric" H 6550 3200 50  0001 C CNN
 F 3 "" H 6550 3200 50  0000 C CNN
 	1    6550 3200
@@
 F 0 "R14" V 3925 4825 50  0000 L CNN
 F 1 "50ohm" V 3975 4700 50  0000 L CNN
-F 2 "Resistor_SMD:R_0402_1005Metric" H 4050 4850 50  0001 C CNN
+F 2 "Resistor_SMD:R_0603_1608Metric" H 4050 4850 50  0001 C CNN
 F 3 "" H 4050 4850 50  0000 C CNN
 	1    4050 4850
@@
 F 0 "R15" V 4125 4925 50  0000 L CNN
 F 1 "50ohm" V 3975 4850 50  0000 L CNN
-F 2 "Resistor_SMD:R_0402_1005Metric" H 4050 5000 50  0001 C CNN
+F 2 "Resistor_SMD:R_0603_1608Metric" H 4050 5000 50  0001 C CNN
 F 3 "" H 4050 5000 50  0000 C CNN
 	1    4050 5000

Commit message: Added 3D models...
25MHz oscillator -> footprint no longer handsoldering variant.
Parts:
- XTAL1: footprint Crystal:Crystal_SMD_3225-4Pin_3.2x2.5mm_HandSoldering -> Crystal:Crystal_SMD_3225-4Pin_3.2x2.5mm
Changed lines of the file:
@@
 F 0 "XTAL1" H 1650 3300 50  0000 L CNN
 F 1 "25MHz 20pF" H 975 3475 50  0000 L CNN
-F 2 "Crystal:Crystal_SMD_3225-4Pin_3.2x2.5mm_HandSoldering" H 1600 3525 50  0001 C CNN
+F 2 "Crystal:Crystal_SMD_3225-4Pin_3.2x2.5mm" H 1600 3525 50  0001 C CNN
 F 3 "" H 1600 3525 50  0001 C CNN
 	1    1600 3525

Commit message: HW rev. 1 - Gerbers
HW: 0406 -> 0603
Parts:
- C17, C18, C19, C20, C21, C22, C23, C24, C25, C26, C27, C28, C29, C30, C31, C32, C33, C34, C35, C36, C37, C38, C39, C40, C41, C42, C54: footprint Capacitor_SMD:C_0402_1005Metric -> Capacitor_SMD:C_0603_1608Metric
- L2, L3, L4, L5, L6, L7: footprint Inductor_SMD:L_0402_1005Metric -> Inductor_SMD:L_0603_1608Metric
- R13, R16: footprint Resistor_SMD:R_0402_1005Metric -> Resistor_SMD:R_0603_1608Metric
Changed lines of the file:
@@
 F 0 "C17" H 1650 6850 50  0000 L CNN
 F 1 "100nF" H 1650 6700 50  0000 L CNN
-F 2 "Capacitor_SMD:C_0402_1005Metric" H 1750 6900 50  0001 C CNN
+F 2 "Capacitor_SMD:C_0603_1608Metric" H 1750 6900 50  0001 C CNN
 F 3 "" H 1750 6900 50  0000 C CNN
 	1    1750 6900
@@
 F 0 "C22" H 1900 6850 50  0000 L CNN
 F 1 "100nF" H 1900 6700 50  0000 L CNN
-F 2 "Capacitor_SMD:C_0402_1005Metric" H 2000 6900 50  0001 C CNN
+F 2 "Capacitor_SMD:C_0603_1608Metric" H 2000 6900 50  0001 C CNN
 F 3 "" H 2000 6900 50  0000 C CNN
 	1    2000 6900
@@
 F 0 "C24" H 2150 6850 50  0000 L CNN
 F 1 "100nF" H 2150 6700 50  0000 L CNN
-F 2 "Capacitor_SMD:C_0402_1005Metric" H 2250 6900 50  0001 C CNN
+F 2 "Capacitor_SMD:C_0603_1608Metric" H 2250 6900 50  0001 C CNN
 F 3 "" H 2250 6900 50  0000 C CNN
 	1    2250 6900
@@
 F 0 "C25" H 2400 6850 50  0000 L CNN
 F 1 "100nF" H 2400 6700 50  0000 L CNN
-F 2 "Capacitor_SMD:C_0402_1005Metric" H 2500 6900 50  0001 C CNN
+F 2 "Capacitor_SMD:C_0603_1608Metric" H 2500 6900 50  0001 C CNN
 F 3 "" H 2500 6900 50  0000 C CNN
 	1    2500 6900
@@
 F 0 "C26" H 2650 6850 50  0000 L CNN
 F 1 "100nF" H 2650 6700 50  0000 L CNN
-F 2 "Capacitor_SMD:C_0402_1005Metric" H 2750 6900 50  0001 C CNN
+F 2 "Capacitor_SMD:C_0603_1608Metric" H 2750 6900 50  0001 C CNN
 F 3 "" H 2750 6900 50  0000 C CNN
 	1    2750 6900
@@
 F 0 "C27" H 2900 6850 50  0000 L CNN
 F 1 "100nF" H 2900 6700 50  0000 L CNN
-F 2 "Capacitor_SMD:C_0402_1005Metric" H 3000 6900 50  0001 C CNN
+F 2 "Capacitor_SMD:C_0603_1608Metric" H 3000 6900 50  0001 C CNN
 F 3 "" H 3000 6900 50  0000 C CNN
 	1    3000 6900
@@
 F 0 "C29" H 3150 6850 50  0000 L CNN
 F 1 "100nF" H 3150 6700 50  0000 L CNN
-F 2 "Capacitor_SMD:C_0402_1005Metric" H 3250 6900 50  0001 C CNN
+F 2 "Capacitor_SMD:C_0603_1608Metric" H 3250 6900 50  0001 C CNN
 F 3 "" H 3250 6900 50  0000 C CNN
 	1    3250 6900
@@
 F 0 "C30" H 3400 6850 50  0000 L CNN
 F 1 "100nF" H 3400 6700 50  0000 L CNN
-F 2 "Capacitor_SMD:C_0402_1005Metric" H 3500 6900 50  0001 C CNN
+F 2 "Capacitor_SMD:C_0603_1608Metric" H 3500 6900 50  0001 C CNN
 F 3 "" H 3500 6900 50  0000 C CNN
 	1    3500 6900
@@
 F 0 "C18" H 1650 7325 50  0000 L CNN
 F 1 "100nF" H 1650 7175 50  0000 L CNN
-F 2 "Capacitor_SMD:C_0402_1005Metric" H 1750 7375 50  0001 C CNN
+F 2 "Capacitor_SMD:C_0603_1608Metric" H 1750 7375 50  0001 C CNN
 F 3 "" H 1750 7375 50  0000 C CNN
 	1    1750 7375
@@
 F 0 "C23" H 1900 7325 50  0000 L CNN
 F 1 "100nF" H 1900 7175 50  0000 L CNN
-F 2 "Capacitor_SMD:C_0402_1005Metric" H 2000 7375 50  0001 C CNN
+F 2 "Capacitor_SMD:C_0603_1608Metric" H 2000 7375 50  0001 C CNN
 F 3 "" H 2000 7375 50  0000 C CNN
 	1    2000 7375
@@
 F 0 "C28" H 3000 7300 50  0000 L CNN
 F 1 "100nF" H 3000 7150 50  0000 L CNN
-F 2 "Capacitor_SMD:C_0402_1005Metric" H 3100 7350 50  0001 C CNN
+F 2 "Capacitor_SMD:C_0603_1608Metric" H 3100 7350 50  0001 C CNN
 F 3 "" H 3100 7350 50  0000 C CNN
 	1    3100 7350
@@
 F 0 "C33" H 6810 3270 50  0000 L CNN
 F 1 "22pF" H 6900 3200 50  0000 L CNN
-F 2 "Capacitor_SMD:C_0402_1005Metric" H 6800 3200 50  0001 C CNN
+F 2 "Capacitor_SMD:C_0603_1608Metric" H 6800 3200 50  0001 C CNN
 F 3 "" H 6800 3200 50  0000 C CNN
 	1    6800 3200
@@
 F 0 "L2" V 6900 3000 50  0000 L CNN
 F 1 "12nH" V 7000 2950 50  0000 L CNN
-F 2 "Inductor_SMD:L_0402_1005Metric" H 6950 3050 50  0001 C CNN
+F 2 "Inductor_SMD:L_0603_1608Metric" H 6950 3050 50  0001 C CNN
 F 3 "" H 6950 3050 50  0000 C CNN
 	1    6950 3050
@@
 F 0 "L3" V 6900 3350 50  0000 L CNN
 F 1 "12nH" V 7000 3250 50  0000 L CNN
-F 2 "Inductor_SMD:L_0402_1005Metric" H 6950 3350 50  0001 C CNN
+F 2 "Inductor_SMD:L_0603_1608Metric" H 6950 3350 50  0001 C CNN
 F 3 "" H 6950 3350 50  0000 C CNN
 	1    6950 3350
@@
 F 0 "C34" V 6900 2900 50  0000 L CNN
 F 1 "39pF" V 7050 2750 50  0000 L CNN
-F 2 "Capacitor_SMD:C_0402_1005Metric" H 6950 2850 50  0001 C CNN
+F 2 "Capacitor_SMD:C_0603_1608Metric" H 6950 2850 50  0001 C CNN
 F 3 "" H 6950 2850 50  0000 C CNN
 	1    6950 2850
@@
 F 0 "C35" V 7000 3600 50  0000 L CNN
 F 1 "39pF" V 6850 3450 50  0000 L CNN
-F 2 "Capacitor_SMD:C_0402_1005Metric" H 6950 3550 50  0001 C CNN
+F 2 "Capacitor_SMD:C_0603_1608Metric" H 6950 3550 50  0001 C CNN
 F 3 "" H 6950 3550 50  0000 C CNN
 	1    6950 3550
@@
 F 0 "C36" H 7110 3270 50  0000 L CNN
 F 1 "33pF" H 7200 3200 50  0000 L CNN
-F 2 "Capacitor_SMD:C_0402_1005Metric" H 7100 3200 50  0001 C CNN
+F 2 "Capacitor_SMD:C_0603_1608Metric" H 7100 3200 50  0001 C CNN
 F 3 "" H 7100 3200 50  0000 C CNN
 	1    7100 3200
@@
 F 0 "L4" V 7200 3000 50  0000 L CNN
 F 1 "18nH" V 7300 2950 50  0000 L CNN
-F 2 "Inductor_SMD:L_0402_1005Metric" H 7250 3050 50  0001 C CNN
+F 2 "Inductor_SMD:L_0603_1608Metric" H 7250 3050 50  0001 C CNN
 F 3 "" H 7250 3050 50  0000 C CNN
 	1    7250 3050
@@
 F 0 "L5" V 7200 3350 50  0000 L CNN
 F 1 "18nH" V 7300 3250 50  0000 L CNN
-F 2 "Inductor_SMD:L_0402_1005Metric" H 7250 3350 50  0001 C CNN
+F 2 "Inductor_SMD:L_0603_1608Metric" H 7250 3350 50  0001 C CNN
 F 3 "" H 7250 3350 50  0000 C CNN
 	1    7250 3350
@@
 F 0 "C37" V 7200 2900 50  0000 L CNN
 F 1 "22pF" V 7350 2750 50  0000 L CNN
-F 2 "Capacitor_SMD:C_0402_1005Metric" H 7250 2850 50  0001 C CNN
+F 2 "Capacitor_SMD:C_0603_1608Metric" H 7250 2850 50  0001 C CNN
 F 3 "" H 7250 2850 50  0000 C CNN
 	1    7250 2850
@@
 F 0 "C38" V 7300 3600 50  0000 L CNN
 F 1 "22pF" V 7150 3450 50  0000 L CNN
-F 2 "Capacitor_SMD:C_0402_1005Metric" H 7250 3550 50  0001 C CNN
+F 2 "Capacitor_SMD:C_0603_1608Metric" H 7250 3550 50  0001 C CNN
 F 3 "" H 7250 3550 50  0000 C CNN
 	1    7250 3550
@@
 F 0 "C39" H 7410 3270 50  0000 L CNN
 F 1 "39pF" H 7500 3200 50  0000 L CNN
-F 2 "Capacitor_SMD:C_0402_1005Metric" H 7400 3200 50  0001 C CNN
+F 2 "Capacitor_SMD:C_0603_1608Metric" H 7400 3200 50  0001 C CNN
 F 3 "" H 7400 3200 50  0000 C CNN
 	1    7400 3200
@@
 F 0 "L6" V 7500 3000 50  0000 L CNN
 F 1 "20nH" V 7600 2950 50  0000 L CNN
-F 2 "Inductor_SMD:L_0402_1005Metric" H 7550 3050 50  0001 C CNN
+F 2 "Inductor_SMD:L_0603_1608Metric" H 7550 3050 50  0001 C CNN
 F 3 "" H 7550 3050 50  0000 C CNN
 	1    7550 3050
@@
 F 0 "L7" V 7500 3350 50  0000 L CNN
 F 1 "20nH" V 7600 3250 50  0000 L CNN
-F 2 "Inductor_SMD:L_0402_1005Metric" H 7550 3350 50  0001 C CNN
+F 2 "Inductor_SMD:L_0603_1608Metric" H 7550 3350 50  0001 C CNN
 F 3 "" H 7550 3350 50  0000 C CNN
 	1    7550 3350
@@
 F 0 "C40" V 7500 2900 50  0000 L CNN
 F 1 "7.5pF" V 7650 2750 50  0000 L CNN
-F 2 "Capacitor_SMD:C_0402_1005Metric" H 7550 2850 50  0001 C CNN
+F 2 "Capacitor_SMD:C_0603_1608Metric" H 7550 2850 50  0001 C CNN
 F 3 "" H 7550 2850 50  0000 C CNN
 	1    7550 2850
@@
 F 0 "C41" V 7600 3600 50  0000 L CNN
 F 1 "7.5pF" V 7450 3450 50  0000 L CNN
-F 2 "Capacitor_SMD:C_0402_1005Metric" H 7550 3550 50  0001 C CNN
+F 2 "Capacitor_SMD:C_0603_1608Metric" H 7550 3550 50  0001 C CNN
 F 3 "" H 7550 3550 50  0000 C CNN
 	1    7550 3550
@@
 F 0 "C42" H 7710 3270 50  0000 L CNN
 F 1 "33pF" H 7800 3200 50  0000 L CNN
-F 2 "Capacitor_SMD:C_0402_1005Metric" H 7700 3200 50  0001 C CNN
+F 2 "Capacitor_SMD:C_0603_1608Metric" H 7700 3200 50  0001 C CNN
 F 3 "" H 7700 3200 50  0000 C CNN
 	1    7700 3200
@@
 F 0 "C32" H 6360 3870 50  0000 L CNN
 F 1 "22pF" H 6450 3800 50  0000 L CNN
-F 2 "Capacitor_SMD:C_0402_1005Metric" H 6350 3800 50  0001 C CNN
+F 2 "Capacitor_SMD:C_0603_1608Metric" H 6350 3800 50  0001 C CNN
 F 3 "" H 6350 3800 50  0000 C CNN
 	1    6350 3800
@@
 F 0 "R16" V 5200 4550 50  0000 L CNN
 F 1 "3.92kohm" V 5050 4350 50  0000 L CNN
-F 2 "Resistor_SMD:R_0402_1005Metric" H 5150 4450 50  0001 C CNN
+F 2 "Resistor_SMD:R_0603_1608Metric" H 5150 4450 50  0001 C CNN
 F 3 "" H 5150 4450 50  0000 C CNN
 	1    5150 4450
@@
 F 0 "C31" H 4810 4620 50  0000 L CNN
 F 1 "1uF" H 4900 4550 50  0000 L CNN
-F 2 "Capacitor_SMD:C_0402_1005Metric" H 4800 4550 50  0001 C CNN
+F 2 "Capacitor_SMD:C_0603_1608Metric" H 4800 4550 50  0001 C CNN
 F 3 "" H 4800 4550 50  0000 C CNN
 	1    4800 4550
@@
 F 0 "C21" H 2010 3730 50  0000 L CNN
 F 1 "39pF" H 2010 3580 50  0000 L CNN
-F 2 "Capacitor_SMD:C_0402_1005Metric" H 2000 3660 50  0001 C CNN
+F 2 "Capacitor_SMD:C_0603_1608Metric" H 2000 3660 50  0001 C CNN
 F 3 "" H 2000 3660 50  0000 C CNN
 	1    2000 3660
@@
 F 0 "C20" H 2010 3355 50  0000 L CNN
 F 1 "39pF" H 2010 3205 50  0000 L CNN
-F 2 "Capacitor_SMD:C_0402_1005Metric" H 2000 3285 50  0001 C CNN
+F 2 "Capacitor_SMD:C_0603_1608Metric" H 2000 3285 50  0001 C CNN
 F 3 "" H 2000 3285 50  0000 C CNN
 	1    2000 3285
@@
 F 0 "C19" H 1910 4420 50  0000 L CNN
 F 1 "10nF" H 1910 4270 50  0000 L CNN
-F 2 "Capacitor_SMD:C_0402_1005Metric" H 1900 4350 50  0001 C CNN
+F 2 "Capacitor_SMD:C_0603_1608Metric" H 1900 4350 50  0001 C CNN
 F 3 "" H 1900 4350 50  0000 C CNN
 	1    1900 4350
@@
 F 0 "R13" H 2230 4370 50  0000 L CNN
 F 1 "243ohm" H 2230 4310 50  0000 L CNN
-F 2 "Resistor_SMD:R_0402_1005Metric" H 2200 4350 50  0001 C CNN
+F 2 "Resistor_SMD:R_0603_1608Metric" H 2200 4350 50  0001 C CNN
 F 3 "" H 2200 4350 50  0000 C CNN
 	1    2200 4350
@@
 F 0 "C54" H 3575 6875 50  0000 L CNN
 F 1 "100nF" H 3575 6725 50  0000 L CNN
-F 2 "Capacitor_SMD:C_0402_1005Metric" H 3675 6925 50  0001 C CNN
+F 2 "Capacitor_SMD:C_0603_1608Metric" H 3675 6925 50  0001 C CNN
 F 3 "" H 3675 6925 50  0000 C CNN
 	1    3675 6925
