File: Hardware/JTAGConn.sch (KiCad schematic (older format))
At the start: 5 parts

Commit message: Second actual HW commit
First finished draft of HW layout and PCB design.
Parts:
- C43: renamed from C56; footprint Capacitors_SMD:C_0805_HandSoldering -> Capacitor_SMD:C_0402_1005Metric
- CON1: renamed from CON?; footprint (none) -> FPC_conn:HFW6R_2STE1LF
- R18: renamed from R20; footprint Resistors_SMD:R_0805_HandSoldering -> Resistor_SMD:R_0402_1005Metric
- R19: renamed from R21; footprint Resistors_SMD:R_0805_HandSoldering -> Resistor_SMD:R_0402_1005Metric
- R20: renamed from R22; footprint Resistors_SMD:R_0805_HandSoldering -> Resistor_SMD:R_0402_1005Metric
Changed lines of the file:
@@
 $EndDescr
 $Comp
-L power:VCC #PWR069
+L power:VCC #PWR052
 U 1 1 58890759
 P 3750 2700
-F 0 "#PWR069" H 3750 2550 50  0001 C CNN
+F 0 "#PWR052" H 3750 2550 50  0001 C CNN
 F 1 "VCC" H 3750 2850 50  0000 C CNN
 F 2 "" H 3750 2700 50  0000 C CNN
@@
 $EndComp
 $Comp
-L Device:R_Small R20
+L Device:R_Small R18
 U 1 1 58890834
 P 3150 2950
-F 0 "R20" H 3180 2970 50  0000 L CNN
+F 0 "R18" H 3180 2970 50  0000 L CNN
 F 1 "100kohm" V 3200 3050 50  0000 L CNN
-F 2 "Resistors_SMD:R_0805_HandSoldering" H 3150 2950 50  0001 C CNN
+F 2 "Resistor_SMD:R_0402_1005Metric" H 3150 2950 50  0001 C CNN
 F 3 "" H 3150 2950 50  0000 C CNN
 	1    3150 2950
@@
 $EndComp
 $Comp
-L Device:R_Small R21
+L Device:R_Small R19
 U 1 1 588908E2
 P 3350 2950
-F 0 "R21" H 3380 2970 50  0000 L CNN
+F 0 "R19" H 3380 2970 50  0000 L CNN
 F 1 "100kohm" V 3400 3050 50  0000 L CNN
-F 2 "Resistors_SMD:R_0805_HandSoldering" H 3350 2950 50  0001 C CNN
+F 2 "Resistor_SMD:R_0402_1005Metric" H 3350 2950 50  0001 C CNN
 F 3 "" H 3350 2950 50  0000 C CNN
 	1    3350 2950
@@
 $EndComp
 $Comp
-L Device:R_Small R22
+L Device:R_Small R20
 U 1 1 588908FF
 P 3550 2950
-F 0 "R22" H 3580 2970 50  0000 L CNN
+F 0 "R20" H 3580 2970 50  0000 L CNN
 F 1 "100kohm" V 3600 3050 50  0000 L CNN
-F 2 "Resistors_SMD:R_0805_HandSoldering" H 3550 2950 50  0001 C CNN
+F 2 "Resistor_SMD:R_0402_1005Metric" H 3550 2950 50  0001 C CNN
 F 3 "" H 3550 2950 50  0000 C CNN
 	1    3550 2950
@@
 Connection ~ 3350 3500
 $Comp
-L Device:C_Small C56
+L Device:C_Small C43
 U 1 1 58890FEC
 P 3250 3950
-F 0 "C56" H 3260 4020 50  0000 L CNN
+F 0 "C43" H 3260 4020 50  0000 L CNN
 F 1 "100nF" H 3260 3870 50  0000 L CNN
-F 2 "Capacitors_SMD:C_0805_HandSoldering" H 3250 3950 50  0001 C CNN
+F 2 "Capacitor_SMD:C_0402_1005Metric" H 3250 3950 50  0001 C CNN
 F 3 "" H 3250 3950 50  0000 C CNN
 	1    3250 3950
@@
 	3250 3850 3250 3700
 $Comp
-L power:GND #PWR068
+L power:GND #PWR050
 U 1 1 58891062
 P 3250 4100
-F 0 "#PWR068" H 3250 3850 50  0001 C CNN
+F 0 "#PWR050" H 3250 3850 50  0001 C CNN
 F 1 "GND" H 3250 3950 50  0000 C CNN
 F 2 "" H 3250 4100 50  0000 C CNN
@@
 	3550 3400 2900 3400
 $Comp
-L fpc_conn:FPC_6POS CON?
+L fpc_conn:FPC_6POS CON1
 U 1 1 5C507911
 P 4200 3800
-F 0 "CON?" H 4277 4103 60  0000 L CNN
+F 0 "CON1" H 4277 4103 60  0000 L CNN
 F 1 "FPC_6POS" H 4277 3997 60  0000 L CNN
-F 2 "" H 4200 3800 60  0001 C CNN
+F 2 "FPC_conn:HFW6R_2STE1LF" H 4200 3800 60  0001 C CNN
 F 3 "" H 4200 3800 60  0001 C CNN
 	1    4200 3800
@@
 Connection ~ 3250 3700
 $Comp
-L power:GND #PWR?
+L power:GND #PWR051
 U 1 1 5C508C3E
 P 3675 4100
-F 0 "#PWR?" H 3675 3850 50  0001 C CNN
+F 0 "#PWR051" H 3675 3850 50  0001 C CNN
 F 1 "GND" H 3675 3950 50  0000 C CNN
 F 2 "" H 3675 4100 50  0000 C CNN

Commit message: HW rev. 1 - Gerbers
HW: 0406 -> 0603
Parts:
- C43: footprint Capacitor_SMD:C_0402_1005Metric -> Capacitor_SMD:C_0603_1608Metric
- R18, R19, R20: footprint Resistor_SMD:R_0402_1005Metric -> Resistor_SMD:R_0603_1608Metric
Changed lines of the file:
@@
 F 0 "R18" H 3180 2970 50  0000 L CNN
 F 1 "100kohm" V 3200 3050 50  0000 L CNN
-F 2 "Resistor_SMD:R_0402_1005Metric" H 3150 2950 50  0001 C CNN
+F 2 "Resistor_SMD:R_0603_1608Metric" H 3150 2950 50  0001 C CNN
 F 3 "" H 3150 2950 50  0000 C CNN
 	1    3150 2950
@@
 F 0 "R19" H 3380 2970 50  0000 L CNN
 F 1 "100kohm" V 3400 3050 50  0000 L CNN
-F 2 "Resistor_SMD:R_0402_1005Metric" H 3350 2950 50  0001 C CNN
+F 2 "Resistor_SMD:R_0603_1608Metric" H 3350 2950 50  0001 C CNN
 F 3 "" H 3350 2950 50  0000 C CNN
 	1    3350 2950
@@
 F 0 "R20" H 3580 2970 50  0000 L CNN
 F 1 "100kohm" V 3600 3050 50  0000 L CNN
-F 2 "Resistor_SMD:R_0402_1005Metric" H 3550 2950 50  0001 C CNN
+F 2 "Resistor_SMD:R_0603_1608Metric" H 3550 2950 50  0001 C CNN
 F 3 "" H 3550 2950 50  0000 C CNN
 	1    3550 2950
@@
 F 0 "C43" H 3260 4020 50  0000 L CNN
 F 1 "100nF" H 3260 3870 50  0000 L CNN
-F 2 "Capacitor_SMD:C_0402_1005Metric" H 3250 3950 50  0001 C CNN
+F 2 "Capacitor_SMD:C_0603_1608Metric" H 3250 3950 50  0001 C CNN
 F 3 "" H 3250 3950 50  0000 C CNN
 	1    3250 3950
