File: Hardware/LCD1602.sch (KiCad schematic (older format))
At the start: 6 parts, among them U6 RC1602A, U7 TXB0108PWR

Commit message: Second actual HW commit
First finished draft of HW layout and PCB design.
Parts:
- C10: renamed from C58; footprint Capacitors_SMD:C_0805_HandSoldering -> Capacitor_SMD:C_0402_1005Metric
- C9: renamed from C57; footprint Capacitors_SMD:C_0805_HandSoldering -> Capacitor_SMD:C_0402_1005Metric
- R11, R12: footprint Resistors_SMD:R_0805_HandSoldering -> Resistor_SMD:R_0402_1005Metric
- U2: renamed from U6; footprint Pin_Headers:Pin_Header_Straight_1x16_Pitch2.54mm -> Connector_PinHeader_2.54mm:PinHeader_1x16_P2.54mm_Vertical
- U3: renamed from U7; footprint Housings_SSOP:TSSOP-20_4.4x6.5mm_Pitch0.65mm -> Package_SO:TSSOP-20_4.4x6.5mm_P0.65mm
Changed lines of the file:
@@
 F 0 "R11" H 4605 3220 50  0000 L CNN
 F 1 "220ohm" H 4605 3160 50  0000 L CNN
-F 2 "Resistors_SMD:R_0805_HandSoldering" H 4575 3200 50  0001 C CNN
+F 2 "Resistor_SMD:R_0402_1005Metric" H 4575 3200 50  0001 C CNN
 F 3 "" H 4575 3200 50  0001 C CNN
 	1    4575 3200
@@
 	4475 3200 4375 3200
 $Comp
-L power:+5V #PWR040
+L power:+5V #PWR026
 U 1 1 59DC44C0
 P 4375 3100
-F 0 "#PWR040" H 4375 2950 50  0001 C CNN
+F 0 "#PWR026" H 4375 2950 50  0001 C CNN
 F 1 "+5V" H 4375 3240 50  0000 C CNN
 F 2 "" H 4375 3100 50  0001 C CNN
@@
 $EndComp
 $Comp
-L power:GND #PWR041
+L power:GND #PWR027
 U 1 1 59DC4529
 P 4825 3300
-F 0 "#PWR041" H 4825 3050 50  0001 C CNN
+F 0 "#PWR027" H 4825 3050 50  0001 C CNN
 F 1 "GND" H 4825 3150 50  0000 C CNN
 F 2 "" H 4825 3300 50  0001 C CNN
@@
 F 0 "R12" H 4630 3720 50  0000 L CNN
 F 1 "2kohm" H 4630 3660 50  0000 L CNN
-F 2 "Resistors_SMD:R_0805_HandSoldering" H 4600 3700 50  0001 C CNN
+F 2 "Resistor_SMD:R_0402_1005Metric" H 4600 3700 50  0001 C CNN
 F 3 "" H 4600 3700 50  0001 C CNN
 	1    4600 3700
@@
 $EndComp
 $Comp
-L power:GND #PWR039
+L power:GND #PWR025
 U 1 1 59DC4939
 P 4350 3725
-F 0 "#PWR039" H 4350 3475 50  0001 C CNN
+F 0 "#PWR025" H 4350 3475 50  0001 C CNN
 F 1 "GND" H 4350 3575 50  0000 C CNN
 F 2 "" H 4350 3725 50  0001 C CNN
@@
 	4500 3700 4350 3700
 $Comp
-L power:GND #PWR043
+L power:GND #PWR029
 U 1 1 59DC4C82
 P 5400 2700
-F 0 "#PWR043" H 5400 2450 50  0001 C CNN
+F 0 "#PWR029" H 5400 2450 50  0001 C CNN
 F 1 "GND" H 5400 2550 50  0000 C CNN
 F 2 "" H 5400 2700 50  0001 C CNN
@@
 	5275 2700 5275 2800
 $Comp
-L power:+5V #PWR042
+L power:+5V #PWR028
 U 1 1 59DC4CDC
 P 5375 4300
-F 0 "#PWR042" H 5375 4150 50  0001 C CNN
+F 0 "#PWR028" H 5375 4150 50  0001 C CNN
 F 1 "+5V" H 5375 4440 50  0000 C CNN
 F 2 "" H 5375 4300 50  0001 C CNN
@@
 NoConn ~ 5925 2775
 $Comp
-L athir:RC1602A U6
+L athir:RC1602A U2
 U 1 1 59DC759C
 P 5275 3500
-F 0 "U6" H 5025 4150 50  0000 C CNN
+F 0 "U2" H 5025 4150 50  0000 C CNN
 F 1 "RC1602A" H 5385 4150 50  0000 L CNN
-F 2 "Pin_Headers:Pin_Header_Straight_1x16_Pitch2.54mm" H 5375 2700 50  0001 C CNN
+F 2 "Connector_PinHeader_2.54mm:PinHeader_1x16_P2.54mm_Vertical" H 5375 2700 50  0001 C CNN
 F 3 "" H 5375 3400 50  0001 C CNN
 	1    5275 3500
@@
 $EndComp
 $Comp
-L Device:C_Small C57
+L Device:C_Small C9
 U 1 1 5B8D3035
 P 4125 5150
-F 0 "C57" H 4217 5196 50  0000 L CNN
+F 0 "C9" H 4217 5196 50  0000 L CNN
 F 1 "0.1uF" H 4217 5105 50  0000 L CNN
-F 2 "Capacitors_SMD:C_0805_HandSoldering" H 4125 5150 50  0001 C CNN
+F 2 "Capacitor_SMD:C_0402_1005Metric" H 4125 5150 50  0001 C CNN
 F 3 "" H 4125 5150 50  0001 C CNN
 	1    4125 5150
@@
 $EndComp
 $Comp
-L athir:TXB0108PWR U7
+L athir:TXB0108PWR U3
 U 1 1 5B8D59AC
 P 5300 5300
-F 0 "U7" H 5300 5967 50  0000 C CNN
+F 0 "U3" H 5300 5967 50  0000 C CNN
 F 1 "TXB0108PWR" H 5300 5876 50  0000 C CNN
-F 2 "Housings_SSOP:TSSOP-20_4.4x6.5mm_Pitch0.65mm" H 5650 5750 50  0001 L CNN
+F 2 "Package_SO:TSSOP-20_4.4x6.5mm_P0.65mm" H 5650 5750 50  0001 L CNN
 F 3 "http://www.ti.com/lit/ds/symlink/txb0108.pdf" H 5300 5200 50  0001 C CNN
 	1    5300 5300
@@
 $EndComp
 $Comp
-L power:+1V8 #PWR0101
+L power:+1V8 #PWR024
 U 1 1 5B8DADA5
 P 4300 4700
-F 0 "#PWR0101" H 4300 4550 50  0001 C CNN
+F 0 "#PWR024" H 4300 4550 50  0001 C CNN
 F 1 "+1V8" H 4300 4840 50  0000 C CNN
 F 2 "" H 4300 4700 50  0001 C CNN
@@
 	4300 5000 4900 5000
 $Comp
-L Device:C_Small C58
+L Device:C_Small C10
 U 1 1 5B8DC34E
 P 6200 5175
-F 0 "C58" H 6292 5221 50  0000 L CNN
+F 0 "C10" H 6292 5221 50  0000 L CNN
 F 1 "0.1uF" H 6292 5130 50  0000 L CNN
-F 2 "Capacitors_SMD:C_0805_HandSoldering" H 6200 5175 50  0001 C CNN
+F 2 "Capacitor_SMD:C_0402_1005Metric" H 6200 5175 50  0001 C CNN
 F 3 "" H 6200 5175 50  0001 C CNN
 	1    6200 5175
@@
 $EndComp
 $Comp
-L power:+5V #PWR0102
+L power:+5V #PWR031
 U 1 1 5B8DC394
 P 6200 4750
-F 0 "#PWR0102" H 6200 4600 50  0001 C CNN
+F 0 "#PWR031" H 6200 4600 50  0001 C CNN
 F 1 "+5V" H 6200 4890 50  0000 C CNN
 F 2 "" H 6200 4750 50  0001 C CNN
@@
 NoConn ~ 5700 5700
 $Comp
-L power:GND #PWR0103
+L power:GND #PWR030
 U 1 1 5B8EAE3C
 P 5800 6125
-F 0 "#PWR0103" H 5800 5875 50  0001 C CNN
+F 0 "#PWR030" H 5800 5875 50  0001 C CNN
 F 1 "GND" H 5800 5975 50  0000 C CNN
 F 2 "" H 5800 6125 50  0001 C CNN

Commit message: HW rev. 1 - Gerbers
HW: 0406 -> 0603
Parts:
- C10, C9: footprint Capacitor_SMD:C_0402_1005Metric -> Capacitor_SMD:C_0603_1608Metric
- R11, R12: footprint Resistor_SMD:R_0402_1005Metric -> Resistor_SMD:R_0603_1608Metric
Changed lines of the file:
@@
 F 0 "R11" H 4605 3220 50  0000 L CNN
 F 1 "220ohm" H 4605 3160 50  0000 L CNN
-F 2 "Resistor_SMD:R_0402_1005Metric" H 4575 3200 50  0001 C CNN
+F 2 "Resistor_SMD:R_0603_1608Metric" H 4575 3200 50  0001 C CNN
 F 3 "" H 4575 3200 50  0001 C CNN
 	1    4575 3200
@@
 F 0 "R12" H 4630 3720 50  0000 L CNN
 F 1 "2kohm" H 4630 3660 50  0000 L CNN
-F 2 "Resistor_SMD:R_0402_1005Metric" H 4600 3700 50  0001 C CNN
+F 2 "Resistor_SMD:R_0603_1608Metric" H 4600 3700 50  0001 C CNN
 F 3 "" H 4600 3700 50  0001 C CNN
 	1    4600 3700
@@
 F 0 "C9" H 4217 5196 50  0000 L CNN
 F 1 "0.1uF" H 4217 5105 50  0000 L CNN
-F 2 "Capacitor_SMD:C_0402_1005Metric" H 4125 5150 50  0001 C CNN
+F 2 "Capacitor_SMD:C_0603_1608Metric" H 4125 5150 50  0001 C CNN
 F 3 "" H 4125 5150 50  0001 C CNN
 	1    4125 5150
@@
 F 0 "C10" H 6292 5221 50  0000 L CNN
 F 1 "0.1uF" H 6292 5130 50  0000 L CNN
-F 2 "Capacitor_SMD:C_0402_1005Metric" H 6200 5175 50  0001 C CNN
+F 2 "Capacitor_SMD:C_0603_1608Metric" H 6200 5175 50  0001 C CNN
 F 3 "" H 6200 5175 50  0001 C CNN
 	1    6200 5175
