File: Hardware/SAMD21PWR.sch (KiCad schematic (older format))
At the start: 7 parts

Commit message: Second actual HW commit
First finished draft of HW layout and PCB design.
Parts:
- C11: renamed from C17; footprint Capacitors_SMD:C_0805_HandSoldering -> Capacitor_SMD:C_0402_1005Metric
- C12: renamed from C18; footprint Capacitors_SMD:C_0805_HandSoldering -> Capacitor_SMD:C_0402_1005Metric
- C13: renamed from C19; footprint Capacitors_SMD:C_0805_HandSoldering -> Capacitor_SMD:C_0402_1005Metric
- C14: renamed from C20; footprint Capacitors_SMD:C_0805_HandSoldering -> Capacitor_SMD:C_0402_1005Metric
- C15: renamed from C21; footprint Capacitors_SMD:C_0805_HandSoldering -> Capacitor_SMD:C_0402_1005Metric
- C16: renamed from C22; footprint Capacitors_SMD:C_0805_HandSoldering -> Capacitor_SMD:C_0402_1005Metric
- L1: footprint Capacitors_SMD:C_0603_HandSoldering -> Capacitor_SMD:C_0603_1608Metric
Changed lines of the file:
@@
 $EndDescr
 $Comp
-L Device:C_Small C21
+L Device:C_Small C15
 U 1 1 588A20B8
 P 4000 1750
-F 0 "C21" H 4010 1820 50  0000 L CNN
+F 0 "C15" H 4010 1820 50  0000 L CNN
 F 1 "100nF" H 4010 1670 50  0000 L CNN
-F 2 "Capacitors_SMD:C_0805_HandSoldering" H 4000 1750 50  0001 C CNN
+F 2 "Capacitor_SMD:C_0402_1005Metric" H 4000 1750 50  0001 C CNN
 F 3 "" H 4000 1750 50  0000 C CNN
 	1    4000 1750
@@
 $EndComp
 $Comp
-L Device:C_Small C19
+L Device:C_Small C13
 U 1 1 588A211B
 P 3700 1750
-F 0 "C19" H 3710 1820 50  0000 L CNN
+F 0 "C13" H 3710 1820 50  0000 L CNN
 F 1 "10uF" H 3710 1670 50  0000 L CNN
-F 2 "Capacitors_SMD:C_0805_HandSoldering" H 3700 1750 50  0001 C CNN
+F 2 "Capacitor_SMD:C_0402_1005Metric" H 3700 1750 50  0001 C CNN
 F 3 "" H 3700 1750 50  0000 C CNN
 	1    3700 1750
@@
 	4650 2050 3450 2050
 $Comp
-L Device:C_Small C18
+L Device:C_Small C12
 U 1 1 588A21C4
 P 3450 2200
-F 0 "C18" H 3460 2270 50  0000 L CNN
+F 0 "C12" H 3460 2270 50  0000 L CNN
 F 1 "100nF" H 3460 2120 50  0000 L CNN
-F 2 "Capacitors_SMD:C_0805_HandSoldering" H 3450 2200 50  0001 C CNN
+F 2 "Capacitor_SMD:C_0402_1005Metric" H 3450 2200 50  0001 C CNN
 F 3 "" H 3450 2200 50  0000 C CNN
 	1    3450 2200
@@
 Connection ~ 3300 2400
 $Comp
-L Device:C_Small C20
+L Device:C_Small C14
 U 1 1 588A22C3
 P 3700 2550
-F 0 "C20" H 3710 2620 50  0000 L CNN
+F 0 "C14" H 3710 2620 50  0000 L CNN
 F 1 "100nF" H 3710 2470 50  0000 L CNN
-F 2 "Capacitors_SMD:C_0805_HandSoldering" H 3700 2550 50  0001 C CNN
+F 2 "Capacitor_SMD:C_0402_1005Metric" H 3700 2550 50  0001 C CNN
 F 3 "" H 3700 2550 50  0000 C CNN
 	1    3700 2550
@@
 VDDCORE
 $Comp
-L Device:C_Small C22
+L Device:C_Small C16
 U 1 1 588A2342
 P 4000 2850
-F 0 "C22" H 4010 2920 50  0000 L CNN
+F 0 "C16" H 4010 2920 50  0000 L CNN
 F 1 "100nF" H 4010 2770 50  0000 L CNN
-F 2 "Capacitors_SMD:C_0805_HandSoldering" H 4000 2850 50  0001 C CNN
+F 2 "Capacitor_SMD:C_0402_1005Metric" H 4000 2850 50  0001 C CNN
 F 3 "" H 4000 2850 50  0000 C CNN
 	1    4000 2850
@@
 Connection ~ 3700 2400
 $Comp
-L power:GND #PWR050
+L power:GND #PWR034
 U 1 1 588A25A6
 P 4650 3000
-F 0 "#PWR050" H 4650 2750 50  0001 C CNN
+F 0 "#PWR034" H 4650 2750 50  0001 C CNN
 F 1 "GND" H 4650 2850 50  0000 C CNN
 F 2 "" H 4650 3000 50  0000 C CNN
@@
 Connection ~ 3700 3000
 $Comp
-L Device:C_Small C17
+L Device:C_Small C11
 U 1 1 588A26A1
 P 3300 2700
-F 0 "C17" H 3310 2770 50  0000 L CNN
+F 0 "C11" H 3310 2770 50  0000 L CNN
 F 1 "10uF" H 3310 2620 50  0000 L CNN
-F 2 "Capacitors_SMD:C_0805_HandSoldering" H 3300 2700 50  0001 C CNN
+F 2 "Capacitor_SMD:C_0402_1005Metric" H 3300 2700 50  0001 C CNN
 F 3 "" H 3300 2700 50  0000 C CNN
 	1    3300 2700
@@
 F 0 "L1" H 3400 1650 45  0000 L BNN
 F 1 "SMD-FERRITE-CHIP-120-OHM-500MA_0603_" H 3500 1700 45  0000 L BNN
-F 2 "Capacitors_SMD:C_0603_HandSoldering" H 3500 1600 60  0001 C CNN
+F 2 "Capacitor_SMD:C_0603_1608Metric" H 3500 1600 60  0001 C CNN
 F 3 "" H 3500 1600 60  0000 C CNN
 F 4 "BLM18AG121SN1D" H 3530 1750 20  0001 C CNN "MPN"
@@
 $EndComp
 $Comp
-L power:+1V8 #PWR048
+L power:+1V8 #PWR032
 U 1 1 58984B17
 P 3300 1500
-F 0 "#PWR048" H 3300 1350 50  0001 C CNN
+F 0 "#PWR032" H 3300 1350 50  0001 C CNN
 F 1 "+1V8" H 3300 1640 50  0000 C CNN
 F 2 "" H 3300 1500 50  0000 C CNN
@@
 $EndComp
 $Comp
-L power:GND #PWR049
+L power:GND #PWR033
 U 1 1 59DD2A76
 P 3700 1900
-F 0 "#PWR049" H 3700 1650 50  0001 C CNN
+F 0 "#PWR033" H 3700 1650 50  0001 C CNN
 F 1 "GND" H 3700 1750 50  0000 C CNN
 F 2 "" H 3700 1900 50  0001 C CNN

Commit message: HW rev. 1 - Gerbers
HW: 0406 -> 0603
Parts:
- C11, C12, C13, C14, C15, C16: footprint Capacitor_SMD:C_0402_1005Metric -> Capacitor_SMD:C_0603_1608Metric
Changed lines of the file:
@@
 F 0 "C15" H 4010 1820 50  0000 L CNN
 F 1 "100nF" H 4010 1670 50  0000 L CNN
-F 2 "Capacitor_SMD:C_0402_1005Metric" H 4000 1750 50  0001 C CNN
+F 2 "Capacitor_SMD:C_0603_1608Metric" H 4000 1750 50  0001 C CNN
 F 3 "" H 4000 1750 50  0000 C CNN
 	1    4000 1750
@@
 F 0 "C13" H 3710 1820 50  0000 L CNN
 F 1 "10uF" H 3710 1670 50  0000 L CNN
-F 2 "Capacitor_SMD:C_0402_1005Metric" H 3700 1750 50  0001 C CNN
+F 2 "Capacitor_SMD:C_0603_1608Metric" H 3700 1750 50  0001 C CNN
 F 3 "" H 3700 1750 50  0000 C CNN
 	1    3700 1750
@@
 F 0 "C12" H 3460 2270 50  0000 L CNN
 F 1 "100nF" H 3460 2120 50  0000 L CNN
-F 2 "Capacitor_SMD:C_0402_1005Metric" H 3450 2200 50  0001 C CNN
+F 2 "Capacitor_SMD:C_0603_1608Metric" H 3450 2200 50  0001 C CNN
 F 3 "" H 3450 2200 50  0000 C CNN
 	1    3450 2200
@@
 F 0 "C14" H 3710 2620 50  0000 L CNN
 F 1 "100nF" H 3710 2470 50  0000 L CNN
-F 2 "Capacitor_SMD:C_0402_1005Metric" H 3700 2550 50  0001 C CNN
+F 2 "Capacitor_SMD:C_0603_1608Metric" H 3700 2550 50  0001 C CNN
 F 3 "" H 3700 2550 50  0000 C CNN
 	1    3700 2550
@@
 F 0 "C16" H 4010 2920 50  0000 L CNN
 F 1 "100nF" H 4010 2770 50  0000 L CNN
-F 2 "Capacitor_SMD:C_0402_1005Metric" H 4000 2850 50  0001 C CNN
+F 2 "Capacitor_SMD:C_0603_1608Metric" H 4000 2850 50  0001 C CNN
 F 3 "" H 4000 2850 50  0000 C CNN
 	1    4000 2850
@@
 F 0 "C11" H 3310 2770 50  0000 L CNN
 F 1 "10uF" H 3310 2620 50  0000 L CNN
-F 2 "Capacitor_SMD:C_0402_1005Metric" H 3300 2700 50  0001 C CNN
+F 2 "Capacitor_SMD:C_0603_1608Metric" H 3300 2700 50  0001 C CNN
 F 3 "" H 3300 2700 50  0000 C CNN
 	1    3300 2700
