File: Hardware/powersheet.sch (KiCad schematic (older format))
At the start: 22 parts

Commit message: Second actual HW commit
First finished draft of HW layout and PCB design.
Parts:
- removed C? (x3): 100nF, Capacitors_SMD:C_0805_HandSoldering, symbol Device:C_Small
- removed C? (x3): 10uF, Capacitors_SMD:C_0805_HandSoldering, symbol Device:C_Small
- removed U?: LD1117S50TR, Common-Parts-Library:LD1117S50TR_SOT230P700X180-4N, symbol Regulator_Linear:LD1117S50TR_SOT223
- removed U?: LD1117S33TR, Common-Parts-Library:LD1117S33TR_SOT230P700X180-4N, symbol Regulator_Linear:LD1117S33TR_SOT223
- removed U? (x2): LD1117S18TR, Common-Parts-Library:LD1117S33TR_SOT230P700X180-4N, symbol Regulator_Linear:LD1117S18TR_SOT223
- added C80: 100nF, Capacitor_SMD:C_0402_1005Metric, symbol Device:C_Small
- added C83: 10uF, Capacitor_SMD:C_0402_1005Metric, symbol Device:C_Small
- added U11, U12: MIC5504-1.8YM5, Package_TO_SOT_SMD:SOT-23-5, symbol Regulator_Linear:MIC5504-1.8YM5
- C76, C77, C78, C79: renamed from C?; footprint (none) -> Capacitor_SMD:C_0402_1005Metric
- C82, C85: renamed from C?; footprint Capacitors_SMD:C_0805_HandSoldering -> Capacitor_SMD:C_0402_1005Metric
- FL1: renamed from FL?; footprint (none) -> athir:ACP3225
- L8: renamed from L?; footprint (none) -> athir:XFL3012
- PSU+1, PSU-1: renamed from W?; footprint Wire_Pads:SolderWirePad_single_SMD_5x10mm -> TestPoint:TestPoint_THTPad_2.0x2.0mm_Drill1.0mm
- R33: renamed from R?; footprint (none) -> Resistor_SMD:R_0402_1005Metric
- gave numbers to parts that had none: 1
Connections:
- net labels removed: +3.3V
- wire segments 92 -> 82

Commit message: Added BOM
Added BOM.csv
Added Micro-USB
Parts:
- C76: footprint Capacitor_SMD:C_0402_1005Metric -> Capacitor_SMD:CP_Elec_6.3x7.7
Changed lines of the file:
@@
 EESchema Schematic File Version 4
+LIBS:rf-receiver-cache
 EELAYER 26 0
 EELAYER END
@@
 F 0 "C76" H 3117 4171 50  0000 L CNN
 F 1 "100uF" H 3117 4080 50  0000 L CNN
-F 2 "Capacitor_SMD:C_0402_1005Metric" H 3025 4125 50  0001 C CNN
+F 2 "Capacitor_SMD:CP_Elec_6.3x7.7" H 3025 4125 50  0001 C CNN
 F 3 "~" H 3025 4125 50  0001 C CNN
 	1    3025 4125
@@
 	2625 4075 2800 4075
 $Comp
-L power:GND #PWR?
+L power:GND #PWR0107
 U 1 1 5C943E0B
 P 4225 4675
-F 0 "#PWR?" H 4225 4425 50  0001 C CNN
+F 0 "#PWR0107" H 4225 4425 50  0001 C CNN
 F 1 "GND" H 4230 4502 50  0000 C CNN
 F 2 "" H 4225 4675 50  0001 C CNN

Commit message: HW PCB changes
Added IBOM
Added extra spacing between 0402 components.
Parts:
- C76: symbol Device:C_Small -> Device:CP_Small
- C78: footprint Capacitor_SMD:C_0402_1005Metric -> Capacitor_SMD:C_0603_1608Metric
- C79: value 22uF -> 100nF
Changed lines of the file:
@@
 	2295 1135 2295 1185
 $Comp
-L Device:C_Small C76
+L Device:CP_Small C76
 U 1 1 5C542B52
 P 3025 4125
@@
 F 0 "C78" H 5417 4271 50  0000 L CNN
 F 1 "22uF" H 5325 4150 50  0000 L CNN
-F 2 "Capacitor_SMD:C_0402_1005Metric" H 5325 4225 50  0001 C CNN
+F 2 "Capacitor_SMD:C_0603_1608Metric" H 5325 4225 50  0001 C CNN
 F 3 "~" H 5325 4225 50  0001 C CNN
 	1    5325 4225
@@
 P 5575 4225
 F 0 "C79" H 5667 4271 50  0000 L CNN
-F 1 "22uF" H 5667 4180 50  0000 L CNN
+F 1 "100nF" H 5667 4180 50  0000 L CNN
 F 2 "Capacitor_SMD:C_0402_1005Metric" H 5575 4225 50  0001 C CNN
 F 3 "~" H 5575 4225 50  0001 C CNN

Commit message: HW rev. 1 - Gerbers
HW: 0406 -> 0603
Parts:
- added C?: CP_Small, symbol Device:CP_Small
- C77, C79, C80, C82, C83, C85: footprint Capacitor_SMD:C_0402_1005Metric -> Capacitor_SMD:C_0603_1608Metric
- R33: footprint Resistor_SMD:R_0402_1005Metric -> Resistor_SMD:R_0603_1608Metric
Changed lines of the file:
@@
 F 0 "C85" H 8710 4570 50  0000 L CNN
 F 1 "10uF" H 8710 4420 50  0000 L CNN
-F 2 "Capacitor_SMD:C_0402_1005Metric" H 8700 4500 50  0001 C CNN
+F 2 "Capacitor_SMD:C_0603_1608Metric" H 8700 4500 50  0001 C CNN
 F 3 "" H 8700 4500 50  0000 C CNN
 	1    8700 4500
@@
 F 0 "C82" H 7585 4570 50  0000 L CNN
 F 1 "100nF" H 7585 4420 50  0000 L CNN
-F 2 "Capacitor_SMD:C_0402_1005Metric" H 7575 4500 50  0001 C CNN
+F 2 "Capacitor_SMD:C_0603_1608Metric" H 7575 4500 50  0001 C CNN
 F 3 "" H 7575 4500 50  0000 C CNN
 	1    7575 4500
@@
 F 0 "C77" H 3467 4171 50  0000 L CNN
 F 1 "100nF" H 3467 4080 50  0000 L CNN
-F 2 "Capacitor_SMD:C_0402_1005Metric" H 3375 4125 50  0001 C CNN
+F 2 "Capacitor_SMD:C_0603_1608Metric" H 3375 4125 50  0001 C CNN
 F 3 "~" H 3375 4125 50  0001 C CNN
 	1    3375 4125
@@
 F 0 "R33" V 5021 4250 50  0000 C CNN
 F 1 "100k" V 4930 4250 50  0000 C CNN
-F 2 "Resistor_SMD:R_0402_1005Metric" H 4825 4250 50  0001 C CNN
+F 2 "Resistor_SMD:R_0603_1608Metric" H 4825 4250 50  0001 C CNN
 F 3 "~" H 4825 4250 50  0001 C CNN
 	1    4825 4250
 	0    -1   -1   0
-$EndComp
-$Comp
-L Device:C_Small C78
-U 1 1 5C5593D3
-P 5325 4225
-F 0 "C78" H 5417 4271 50  0000 L CNN
-F 1 "22uF" H 5325 4150 50  0000 L CNN
-F 2 "Capacitor_SMD:C_0603_1608Metric" H 5325 4225 50  0001 C CNN
-F 3 "~" H 5325 4225 50  0001 C CNN
-	1    5325 4225
-	1    0    0    -1
 $EndComp
 Wire Wire Line
@@
 F 0 "C79" H 5667 4271 50  0000 L CNN
 F 1 "100nF" H 5667 4180 50  0000 L CNN
-F 2 "Capacitor_SMD:C_0402_1005Metric" H 5575 4225 50  0001 C CNN
+F 2 "Capacitor_SMD:C_0603_1608Metric" H 5575 4225 50  0001 C CNN
 F 3 "~" H 5575 4225 50  0001 C CNN
 	1    5575 4225
@@
 F 0 "C83" H 8610 5645 50  0000 L CNN
 F 1 "10uF" H 8610 5495 50  0000 L CNN
-F 2 "Capacitor_SMD:C_0402_1005Metric" H 8600 5575 50  0001 C CNN
+F 2 "Capacitor_SMD:C_0603_1608Metric" H 8600 5575 50  0001 C CNN
 F 3 "" H 8600 5575 50  0000 C CNN
 	1    8600 5575
@@
 F 0 "C80" H 7485 5645 50  0000 L CNN
 F 1 "100nF" H 7485 5495 50  0000 L CNN
-F 2 "Capacitor_SMD:C_0402_1005Metric" H 7475 5575 50  0001 C CNN
+F 2 "Capacitor_SMD:C_0603_1608Metric" H 7475 5575 50  0001 C CNN
 F 3 "" H 7475 5575 50  0000 C CNN
 	1    7475 5575
@@
 Wire Wire Line
 	4225 4650 4225 4675
+$Comp
+L Device:CP_Small C?
+U 1 1 5C9CC4C1
+P 5975 3950
+F 0 "C?" H 6063 3996 50  0000 L CNN
+F 1 "CP_Small" H 6063 3905 50  0000 L CNN
+F 2 "" H 5975 3950 50  0001 C CNN
+F 3 "~" H 5975 3950 50  0001 C CNN
+	1    5975 3950
+	1    0    0    -1
+$EndComp
+$Comp
+L Device:C_Small C78
+U 1 1 5C5593D3
+P 5325 4225
+F 0 "C78" H 5417 4271 50  0000 L CNN
+F 1 "22uF" H 5325 4150 50  0000 L CNN
+F 2 "Capacitor_SMD:C_0603_1608Metric" H 5325 4225 50  0001 C CNN
+F 3 "~" H 5325 4225 50  0001 C CNN
+	1    5325 4225
+	1    0    0    -1
+$EndComp
 $EndSCHEMATC
