File: Hardware/tayloesheet.sch (KiCad schematic (older format))
At the start: 68 parts, among them IC1 74LVC74, J1 Conn_Coaxial, J2 Conn_Coaxial, J3 Conn_Coaxial, J4 Conn_Coaxial, J5 Audio-Jack-4, J6 Barrel_Jack, U1 LD1117S33TR, U2 OPA300, U3 74LS00, U4 Transformer, U5 74CBTLV3253, U6 NE5532

Commit message: Second actual HW commit
First finished draft of HW layout and PCB design.
Parts:
- removed C1: 100nF, Capacitors_SMD:C_0805_HandSoldering, symbol Device:C_Small
- removed C11, C16, C7: 10uF, Capacitors_SMD:C_0805_HandSoldering, symbol Device:C_Small
- removed C12: 10nF, Capacitors_SMD:C_0805_HandSoldering, symbol Device:C_Small
- removed C15: 1000pF, Capacitors_SMD:C_0805_HandSoldering, symbol Device:C_Small
- removed J1, J3, J4: Conn_Coaxial, Connectors_TE-Connectivity:BNC_Socket_TYCO-AMP_LargePads, symbol Connector:Conn_Coaxial
- removed J5: Audio-Jack-4, athir:SJ1-35235, symbol Connector:AudioJack4_Ground
- removed J6: Barrel_Jack, Connectors:Barrel_Jack_CUI_PJ-102AH, symbol Connector:Barrel_Jack
- removed JP1: DRV_VS_DIRECT, Pin_Headers:Pin_Header_Straight_1x03_Pitch2.54mm, symbol Device:Jumper_NC_Dual
- removed JP2: CLK_DRV_EN, Pin_Headers:Pin_Header_Straight_1x02_Pitch2.54mm, symbol Device:Jumper_NC_Small
- removed R8: 22kOhm, Resistors_SMD:R_0805_HandSoldering, symbol Device:R_Small
- removed TP1, TP2: Test_Point, Wire_Pads:SolderWirePad_single_1mmDrill, symbol Connector:TestPoint
- removed U1: LD1117S33TR, TO_SOT_Packages_SMD:SOT-223, symbol Regulator_Linear:LD1117S33TR_SOT223
- removed U3: 74LS00, Housings_SOIC:SOIC-14_3.9x8.7mm_Pitch1.27mm, symbol 74xx:74LS00
- added C44: 100nF, Capacitor_SMD:C_0402_1005Metric, symbol Device:C_Small
- added C50: 10uF, Capacitor_SMD:C_0402_1005Metric, symbol Device:C_Small
- added J6: AudioJack3_Ground, symbol Connector:AudioJack3_Ground
- added U4: MIC5504-3.3YM5, Package_TO_SOT_SMD:SOT-23-5, symbol Regulator_Linear:MIC5504-3.3YM5
- C45: renamed from C2; footprint Capacitors_SMD:C_0805_HandSoldering -> Capacitor_SMD:C_0402_1005Metric
- C46: renamed from C3; footprint Capacitors_SMD:C_0805_HandSoldering -> Capacitor_SMD:C_0402_1005Metric
- C47: renamed from C4; footprint Capacitors_SMD:C_0805_HandSoldering -> Capacitor_SMD:C_0402_1005Metric
- C48: renamed from C5; footprint Capacitors_SMD:C_0805_HandSoldering -> Capacitor_SMD:C_0402_1005Metric
- C49: renamed from C6; footprint Capacitors_SMD:C_0805_HandSoldering -> Capacitor_SMD:C_0402_1005Metric
- C51: renamed from C8; footprint Capacitors_SMD:C_0805_HandSoldering -> Capacitor_SMD:C_0402_1005Metric
- C52: renamed from C9; footprint Capacitors_SMD:C_0805_HandSoldering -> Capacitor_SMD:C_0402_1005Metric
- C53: renamed from C10; footprint Capacitors_SMD:C_0805_HandSoldering -> Capacitor_SMD:C_0402_1005Metric
- C56: renamed from C13; footprint Capacitors_SMD:C_0805_HandSoldering -> Capacitor_SMD:C_0402_1005Metric
- C57: renamed from C14; footprint Capacitors_SMD:C_0805_HandSoldering -> Capacitor_SMD:C_0402_1005Metric
- C59: renamed from C32; footprint Capacitors_SMD:C_0805_HandSoldering -> Capacitor_SMD:C_0402_1005Metric
- C61: renamed from C17; footprint Capacitors_SMD:C_0805_HandSoldering -> Capacitor_SMD:C_0402_1005Metric
- C62: renamed from C18; footprint Capacitors_SMD:C_0805_HandSoldering -> Capacitor_SMD:C_0402_1005Metric
- C63: renamed from C19; footprint Capacitors_SMD:C_0805_HandSoldering -> Capacitor_SMD:C_0402_1005Metric
- C64: renamed from C20; footprint Capacitors_SMD:C_0805_HandSoldering -> Capacitor_SMD:C_0402_1005Metric
- C65: renamed from C21; footprint Capacitors_SMD:C_0805_HandSoldering -> Capacitor_SMD:C_0402_1005Metric
- C66: renamed from C22; footprint Capacitors_SMD:C_0805_HandSoldering -> Capacitor_SMD:C_0402_1005Metric
- C67: renamed from C23; footprint Capacitors_SMD:C_0805_HandSoldering -> Capacitor_SMD:C_0402_1005Metric
- C68: renamed from C24; footprint Capacitors_SMD:C_0805_HandSoldering -> Capacitor_SMD:C_0402_1005Metric
- C69: renamed from C25; footprint Capacitors_SMD:C_0805_HandSoldering -> Capacitor_SMD:C_0402_1005Metric
- C70: renamed from C26; footprint Capacitors_SMD:C_0805_HandSoldering -> Capacitor_SMD:C_0402_1005Metric
- C71: renamed from C27; footprint Capacitors_SMD:C_0805_HandSoldering -> Capacitor_SMD:C_0402_1005Metric
- C72: renamed from C28; footprint Capacitors_SMD:C_0805_HandSoldering -> Capacitor_SMD:C_0402_1005Metric
- C73: renamed from C29; footprint Capacitors_SMD:C_0805_HandSoldering -> Capacitor_SMD:C_0402_1005Metric
- C74: renamed from C30; footprint Capacitors_SMD:C_0805_HandSoldering -> Capacitor_SMD:C_0402_1005Metric
- C75: renamed from C31; footprint Capacitors_SMD:C_0805_HandSoldering -> Capacitor_SMD:C_0402_1005Metric
- IC3: renamed from IC1; footprint Housings_SOIC:SOIC-14_3.9x8.7mm_Pitch1.27mm -> Package_SO:SOIC-14_3.9x8.7mm_P1.27mm
- J2: footprint Connectors_TE-Connectivity:BNC_Socket_TYCO-AMP_LargePads -> Connector_Coaxial:SMA_Molex_73251-1153_EdgeMount_Horizontal
- R21: renamed from R1; footprint Resistors_SMD:R_0805_HandSoldering -> Resistor_SMD:R_0402_1005Metric
- R22: renamed from R2; footprint Resistors_SMD:R_0805_HandSoldering -> Resistor_SMD:R_0402_1005Metric
- R23: renamed from R3; footprint Resistors_SMD:R_0805_HandSoldering -> Resistor_SMD:R_0402_1005Metric
- R24: renamed from R4; footprint Resistors_SMD:R_0805_HandSoldering -> Resistor_SMD:R_0402_1005Metric
- R25: renamed from R5; footprint Resistors_SMD:R_0805_HandSoldering -> Resistor_SMD:R_0402_1005Metric
- R26: renamed from R6; footprint Resistors_SMD:R_0805_HandSoldering -> Resistor_SMD:R_0402_1005Metric
- R27: renamed from R7; footprint Resistors_SMD:R_0805_HandSoldering -> Resistor_SMD:R_0402_1005Metric
- R29: renamed from R9; footprint Resistors_SMD:R_0805_HandSoldering -> Resistor_SMD:R_0402_1005Metric
- R30: renamed from R10; footprint Resistors_SMD:R_0805_HandSoldering -> Resistor_SMD:R_0402_1005Metric
- R31: renamed from R11; footprint Resistors_SMD:R_0805_HandSoldering -> Resistor_SMD:R_0402_1005Metric
- R32: renamed from R12; footprint Resistors_SMD:R_0805_HandSoldering -> Resistor_SMD:R_0402_1005Metric
- TP3: renamed from TP5; footprint Connectors_TestPoints:Test_Point_Pad_d4.0mm -> TestPoint:TestPoint_Pad_D1.0mm
- TP4: renamed from TP6; footprint Connectors_TestPoints:Test_Point_Pad_d4.0mm -> TestPoint:TestPoint_Pad_D1.0mm
- TP5: renamed from TP3; footprint Connectors_TestPoints:Test_Point_Pad_d4.0mm -> TestPoint:TestPoint_Pad_D1.0mm
- TP6: renamed from TP7; footprint Connectors_TestPoints:Test_Point_Pad_d4.0mm -> TestPoint:TestPoint_Pad_D1.0mm
- TP7: renamed from TP8; footprint Connectors_TestPoints:Test_Point_Pad_d4.0mm -> TestPoint:TestPoint_Pad_D1.0mm
- TP8: renamed from TP4; footprint Connectors_TestPoints:Test_Point_Pad_d4.0mm -> TestPoint:TestPoint_Pad_D1.0mm
- U5: renamed from U2; footprint TO_SOT_Packages_SMD:SOT-23-6_Handsoldering -> Package_TO_SOT_SMD:SOT-23-6_Handsoldering
- U8: renamed from U6; footprint Housings_SOIC:SOIC-8_3.9x4.9mm_Pitch1.27mm -> Package_SO:SOIC-8_3.9x4.9mm_P1.27mm
- U8: renamed from U?; footprint Housings_SOIC:SOIC-8_3.9x4.9mm_Pitch1.27mm -> Package_SO:SOIC-8_3.9x4.9mm_P1.27mm
- U9: renamed from U5; footprint Housings_SSOP:TSSOP-16_4.4x5mm_Pitch0.65mm -> Package_SO:SSOP-16_4.4x5.2mm_P0.65mm
- renumbered U4 to U7
Connections:
- net labels added: +5V
- net labels removed: +3V3, CLK_DRV, VCC, VOUT_N, VOUT_P
- wire segments 341 -> 280
- no-connect marks 3 -> 0

Commit message: Added BOM
Added BOM.csv
Added Micro-USB
Parts:
- removed J6: AudioJack3_Ground, symbol Connector:AudioJack3_Ground
- added J1: Conn_01x05_Female, athir:SJ1-35235, symbol Connector:Conn_01x05_Female
- C52: footprint Capacitor_SMD:C_0402_1005Metric -> Capacitor_SMD:CP_Elec_6.3x7.7
- J2: footprint Connector_Coaxial:SMA_Molex_73251-1153_EdgeMount_Horizontal -> Connector_Coaxial:SMA_Amphenol_132289_EdgeMount
Connections:
- no-connect marks 0 -> 1
Changed lines of the file:
@@
 EESchema Schematic File Version 4
+LIBS:rf-receiver-cache
 EELAYER 26 0
 EELAYER END
@@
 F 0 "C52" H 4475 4975 50  0000 L CNN
 F 1 "47uF" H 4475 4775 50  0000 L CNN
-F 2 "Capacitor_SMD:C_0402_1005Metric" H 4488 4725 50  0001 C CNN
+F 2 "Capacitor_SMD:CP_Elec_6.3x7.7" H 4488 4725 50  0001 C CNN
 F 3 "" H 4450 4875 50  0000 C CNN
 	1    4450 4875
@@
 F 0 "J2" H 2049 651 50  0000 L CNN
 F 1 "Conn_Coaxial" H 2049 560 50  0000 L CNN
-F 2 "Connector_Coaxial:SMA_Molex_73251-1153_EdgeMount_Horizontal" H 1950 675 50  0001 C CNN
+F 2 "Connector_Coaxial:SMA_Amphenol_132289_EdgeMount" H 1950 675 50  0001 C CNN
 F 3 "" H 1950 675 50  0001 C CNN
 	1    1950 675
@@
 L power:GND #PWR080
 U 1 1 5A247566
-P 5100 1550
-F 0 "#PWR080" H 5100 1300 50  0001 C CNN
-F 1 "GND" H 5105 1377 50  0000 C CNN
-F 2 "" H 5100 1550 50  0001 C CNN
-F 3 "" H 5100 1550 50  0001 C CNN
-	1    5100 1550
-	1    0    0    -1
-$EndComp
-Text Label 5300 1225 2    60   ~ 0
+P 4425 1600
+F 0 "#PWR080" H 4425 1350 50  0001 C CNN
+F 1 "GND" H 4430 1427 50  0000 C CNN
+F 2 "" H 4425 1600 50  0001 C CNN
+F 3 "" H 4425 1600 50  0001 C CNN
+	1    4425 1600
+	1    0    0    -1
+$EndComp
+Text Label 4250 1475 0    60   ~ 0
 Q_OUT
-Text Label 5300 1125 2    60   ~ 0
+Text Label 4250 1375 0    60   ~ 0
 I_OUT
 $Comp
@@
 	3350 3090 3350 3110
 Wire Wire Line
-	5025 1225 5300 1225
-Wire Wire Line
-	5025 1125 5300 1125
-Wire Wire Line
 	1950 900  1950 875
 Wire Wire Line
@@
 Wire Wire Line
 	7470 3800 7470 3810
-Wire Wire Line
-	5100 1325 5025 1325
 Wire Wire Line
 	2310 4660 2310 4675
@@
 Wire Wire Line
 	2690 2890 3180 2890
-$Comp
-L Connector:AudioJack3_Ground J6
-U 1 1 5C6F608C
-P 4825 1225
-F 0 "J6" H 4829 1567 50  0000 C CNN
-F 1 "AudioJack3_Ground" H 4829 1476 50  0000 C CNN
-F 2 "" H 4825 1225 50  0001 C CNN
-F 3 "~" H 4825 1225 50  0001 C CNN
-	1    4825 1225
-	1    0    0    -1
-$EndComp
-Wire Wire Line
-	5100 1325 5100 1550
 $Comp
 L power:+3.3V #PWR?
@@
 Wire Wire Line
 	1900 6925 1900 7050
+$Comp
+L Connector:Conn_01x05_Female J1
+U 1 1 5C4A7415
+P 4050 1375
+F 0 "J1" H 3944 950 50  0000 C CNN
+F 1 "Conn_01x05_Female" H 3944 1041 50  0000 C CNN
+F 2 "athir:SJ1-35235" H 4050 1375 50  0001 C CNN
+F 3 "~" H 4050 1375 50  0001 C CNN
+	1    4050 1375
+	-1   0    0    1
+$EndComp
+Wire Wire Line
+	4425 1600 4425 1575
+Wire Wire Line
+	4425 1575 4250 1575
+NoConn ~ 4250 1175
+Wire Wire Line
+	4250 1275 4425 1275
+Wire Wire Line
+	4425 1275 4425 1575
+Connection ~ 4425 1575
 $EndSCHEMATC

Commit message: HW PCB changes
Added IBOM
Added extra spacing between 0402 components.
Parts:
- C64: footprint Capacitor_SMD:C_0402_1005Metric -> Capacitor_SMD:C_0603_1608Metric
- R21, R25: footprint Resistor_SMD:R_0402_1005Metric -> Resistor_SMD:R_0603_1608Metric
- R26, R27: value 2.2k ohm -> 2k ohm
- U9: footprint Package_SO:SSOP-16_4.4x5.2mm_P0.65mm -> Package_SO:TSSOP-16_4.4x5mm_P0.65mm
Changed lines of the file:
@@
 P 4220 4665
 F 0 "R26" V 4310 4635 50  0000 L CNN
-F 1 "2.2k ohm" V 4150 4575 50  0000 L CNN
+F 1 "2k ohm" V 4150 4575 50  0000 L CNN
 F 2 "Resistor_SMD:R_0402_1005Metric" H 4220 4665 50  0001 C CNN
 F 3 "" H 4220 4665 50  0000 C CNN
@@
 P 4720 4885
 F 0 "R27" H 4750 4905 50  0000 L CNN
-F 1 "2.2k ohm" H 4750 4845 50  0000 L CNN
+F 1 "2k ohm" H 4750 4845 50  0000 L CNN
 F 2 "Resistor_SMD:R_0402_1005Metric" H 4720 4885 50  0001 C CNN
 F 3 "" H 4720 4885 50  0000 C CNN
@@
 F 0 "U9" H 8505 4110 50  0000 C CNN
 F 1 "74CBTLV3253" H 8255 5310 50  0000 C CNN
-F 2 "Package_SO:SSOP-16_4.4x5.2mm_P0.65mm" H 9715 3860 50  0001 C CNN
+F 2 "Package_SO:TSSOP-16_4.4x5mm_P0.65mm" H 9715 3860 50  0001 C CNN
 F 3 "" H 9715 3860 50  0000 C CNN
 	1    8555 4560
@@
 F 0 "C64" V 7880 875 50  0000 L CNN
 F 1 "10uF" V 7890 630 50  0000 L CNN
-F 2 "Capacitor_SMD:C_0402_1005Metric" H 7840 850 50  0001 C CNN
+F 2 "Capacitor_SMD:C_0603_1608Metric" H 7840 850 50  0001 C CNN
 F 3 "" H 7840 850 50  0001 C CNN
 	1    7840 850
@@
 F 0 "R21" V 1360 4410 50  0000 L CNN
 F 1 "50ohm" V 1510 4310 50  0000 L CNN
-F 2 "Resistor_SMD:R_0402_1005Metric" H 1435 4460 50  0001 C CNN
+F 2 "Resistor_SMD:R_0603_1608Metric" H 1435 4460 50  0001 C CNN
 F 3 "" H 1435 4460 50  0001 C CNN
 	1    1435 4460
@@
 F 0 "R25" V 2670 4320 50  0000 L CNN
 F 1 "50ohm" V 2885 4210 50  0000 L CNN
-F 2 "Resistor_SMD:R_0402_1005Metric" H 2810 4360 50  0001 C CNN
+F 2 "Resistor_SMD:R_0603_1608Metric" H 2810 4360 50  0001 C CNN
 F 3 "" H 2810 4360 50  0001 C CNN
 	1    2810 4360

Commit message: HW rev. 1 - Gerbers
HW: 0406 -> 0603
Parts:
- C44, C45, C46, C47, C48, C49, C50, C51, C53, C56, C57, C59, C61, C62, C63, C65, C66, C67, C68, C69, C70, C71, C72, C73, C74, C75: footprint Capacitor_SMD:C_0402_1005Metric -> Capacitor_SMD:C_0603_1608Metric
- R22, R23, R24, R26, R27, R29, R30, R31, R32: footprint Resistor_SMD:R_0402_1005Metric -> Resistor_SMD:R_0603_1608Metric
Changed lines of the file:
@@
 F 0 "R26" V 4310 4635 50  0000 L CNN
 F 1 "2k ohm" V 4150 4575 50  0000 L CNN
-F 2 "Resistor_SMD:R_0402_1005Metric" H 4220 4665 50  0001 C CNN
+F 2 "Resistor_SMD:R_0603_1608Metric" H 4220 4665 50  0001 C CNN
 F 3 "" H 4220 4665 50  0000 C CNN
 	1    4220 4665
@@
 F 0 "R27" H 4750 4905 50  0000 L CNN
 F 1 "2k ohm" H 4750 4845 50  0000 L CNN
-F 2 "Resistor_SMD:R_0402_1005Metric" H 4720 4885 50  0001 C CNN
+F 2 "Resistor_SMD:R_0603_1608Metric" H 4720 4885 50  0001 C CNN
 F 3 "" H 4720 4885 50  0000 C CNN
 	1    4720 4885
@@
 F 0 "C53" H 4515 2540 50  0000 L CNN
 F 1 "0.1uF" H 4475 2410 50  0000 L CNN
-F 2 "Capacitor_SMD:C_0402_1005Metric" H 4465 2490 50  0001 C CNN
+F 2 "Capacitor_SMD:C_0603_1608Metric" H 4465 2490 50  0001 C CNN
 F 3 "" H 4465 2490 50  0000 C CNN
 	1    4465 2490
@@
 F 0 "C63" H 7645 3980 50  0000 L CNN
 F 1 "0.1uF" H 7645 3830 50  0000 L CNN
-F 2 "Capacitor_SMD:C_0402_1005Metric" H 7635 3910 50  0001 C CNN
+F 2 "Capacitor_SMD:C_0603_1608Metric" H 7635 3910 50  0001 C CNN
 F 3 "" H 7635 3910 50  0000 C CNN
 	1    7635 3910
@@
 F 0 "C66" H 9010 4470 50  0000 L CNN
 F 1 "40nF" H 9010 4320 50  0000 L CNN
-F 2 "Capacitor_SMD:C_0402_1005Metric" H 9000 4400 50  0001 C CNN
+F 2 "Capacitor_SMD:C_0603_1608Metric" H 9000 4400 50  0001 C CNN
 F 3 "" H 9000 4400 50  0000 C CNN
 	1    9000 4400
@@
 F 0 "C68" H 9210 4470 50  0000 L CNN
 F 1 "40nF" H 9210 4320 50  0000 L CNN
-F 2 "Capacitor_SMD:C_0402_1005Metric" H 9200 4400 50  0001 C CNN
+F 2 "Capacitor_SMD:C_0603_1608Metric" H 9200 4400 50  0001 C CNN
 F 3 "" H 9200 4400 50  0000 C CNN
 	1    9200 4400
@@
 F 0 "C70" H 9410 4470 50  0000 L CNN
 F 1 "40nF" H 9410 4320 50  0000 L CNN
-F 2 "Capacitor_SMD:C_0402_1005Metric" H 9400 4400 50  0001 C CNN
+F 2 "Capacitor_SMD:C_0603_1608Metric" H 9400 4400 50  0001 C CNN
 F 3 "" H 9400 4400 50  0000 C CNN
 	1    9400 4400
@@
 F 0 "C72" H 9610 4470 50  0000 L CNN
 F 1 "40nF" H 9610 4320 50  0000 L CNN
-F 2 "Capacitor_SMD:C_0402_1005Metric" H 9600 4400 50  0001 C CNN
+F 2 "Capacitor_SMD:C_0603_1608Metric" H 9600 4400 50  0001 C CNN
 F 3 "" H 9600 4400 50  0000 C CNN
 	1    9600 4400
@@
 F 0 "R29" V 7525 1825 50  0000 L CNN
 F 1 "10kohm" V 7650 1575 50  0000 L CNN
-F 2 "Resistor_SMD:R_0402_1005Metric" H 7575 1725 50  0001 C CNN
+F 2 "Resistor_SMD:R_0603_1608Metric" H 7575 1725 50  0001 C CNN
 F 3 "" H 7575 1725 50  0001 C CNN
 	1    7575 1725
@@
 F 0 "C56" H 5520 4080 50  0000 L CNN
 F 1 "10uF" H 5520 3930 50  0000 L CNN
-F 2 "Capacitor_SMD:C_0402_1005Metric" H 5510 4010 50  0001 C CNN
+F 2 "Capacitor_SMD:C_0603_1608Metric" H 5510 4010 50  0001 C CNN
 F 3 "" H 5510 4010 50  0001 C CNN
 	1    5510 4010
@@
 F 0 "C61" H 7580 2195 50  0000 L CNN
 F 1 "0.8nF" V 7625 1885 50  0000 L CNN
-F 2 "Capacitor_SMD:C_0402_1005Metric" H 7570 2125 50  0001 C CNN
+F 2 "Capacitor_SMD:C_0603_1608Metric" H 7570 2125 50  0001 C CNN
 F 3 "" H 7570 2125 50  0001 C CNN
 	1    7570 2125
@@
 F 0 "R30" V 7525 2025 50  0000 L CNN
 F 1 "10kohm" V 7650 1775 50  0000 L CNN
-F 2 "Resistor_SMD:R_0402_1005Metric" H 7575 1925 50  0001 C CNN
+F 2 "Resistor_SMD:R_0603_1608Metric" H 7575 1925 50  0001 C CNN
 F 3 "" H 7575 1925 50  0001 C CNN
 	1    7575 1925
@@
 F 0 "R31" V 9600 1850 50  0000 L CNN
 F 1 "10kohm" V 9725 1600 50  0000 L CNN
-F 2 "Resistor_SMD:R_0402_1005Metric" H 9650 1750 50  0001 C CNN
+F 2 "Resistor_SMD:R_0603_1608Metric" H 9650 1750 50  0001 C CNN
 F 3 "" H 9650 1750 50  0001 C CNN
 	1    9650 1750
@@
 F 0 "C73" V 9690 2180 50  0000 L CNN
 F 1 "0.8nF" V 9610 2175 50  0000 L CNN
-F 2 "Capacitor_SMD:C_0402_1005Metric" H 9650 2150 50  0001 C CNN
+F 2 "Capacitor_SMD:C_0603_1608Metric" H 9650 2150 50  0001 C CNN
 F 3 "" H 9650 2150 50  0001 C CNN
 	1    9650 2150
@@
 F 0 "R32" V 9600 2050 50  0000 L CNN
 F 1 "10kohm" V 9725 1800 50  0000 L CNN
-F 2 "Resistor_SMD:R_0402_1005Metric" H 9650 1950 50  0001 C CNN
+F 2 "Resistor_SMD:R_0603_1608Metric" H 9650 1950 50  0001 C CNN
 F 3 "" H 9650 1950 50  0001 C CNN
 	1    9650 1950
@@
 F 0 "C57" H 5820 4080 50  0000 L CNN
 F 1 "10nF" H 5820 3930 50  0000 L CNN
-F 2 "Capacitor_SMD:C_0402_1005Metric" H 5810 4010 50  0001 C CNN
+F 2 "Capacitor_SMD:C_0603_1608Metric" H 5810 4010 50  0001 C CNN
 F 3 "" H 5810 4010 50  0001 C CNN
 	1    5810 4010
@@
 F 0 "R23" V 1535 4810 50  0000 L CNN
 F 1 "10kohm" V 1660 4560 50  0000 L CNN
-F 2 "Resistor_SMD:R_0402_1005Metric" H 1585 4710 50  0001 C CNN
+F 2 "Resistor_SMD:R_0603_1608Metric" H 1585 4710 50  0001 C CNN
 F 3 "" H 1585 4710 50  0001 C CNN
 	1    1585 4710
@@
 F 0 "C46" H 1770 4800 50  0000 L CNN
 F 1 "10uF" H 1670 4675 50  0000 L CNN
-F 2 "Capacitor_SMD:C_0402_1005Metric" H 1760 4730 50  0001 C CNN
+F 2 "Capacitor_SMD:C_0603_1608Metric" H 1760 4730 50  0001 C CNN
 F 3 "" H 1760 4730 50  0001 C CNN
 	1    1760 4730
@@
 F 0 "R22" H 1485 4210 50  0000 L CNN
 F 1 "10kohm" V 1660 3935 50  0000 L CNN
-F 2 "Resistor_SMD:R_0402_1005Metric" H 1585 4085 50  0001 C CNN
+F 2 "Resistor_SMD:R_0603_1608Metric" H 1585 4085 50  0001 C CNN
 F 3 "" H 1585 4085 50  0001 C CNN
 	1    1585 4085
@@
 F 0 "C49" H 1835 4165 50  0000 L CNN
 F 1 "10uF" H 1735 4040 50  0000 L CNN
-F 2 "Capacitor_SMD:C_0402_1005Metric" H 1935 4090 50  0001 C CNN
+F 2 "Capacitor_SMD:C_0603_1608Metric" H 1935 4090 50  0001 C CNN
 F 3 "" H 1935 4090 50  0001 C CNN
 	1    1935 4090
@@
 F 0 "C45" V 1110 4485 50  0000 L CNN
 F 1 "10nF" V 1260 4335 50  0000 L CNN
-F 2 "Capacitor_SMD:C_0402_1005Metric" H 1160 4460 50  0001 C CNN
+F 2 "Capacitor_SMD:C_0603_1608Metric" H 1160 4460 50  0001 C CNN
 F 3 "" H 1160 4460 50  0001 C CNN
 	1    1160 4460
@@
 F 0 "R24" V 2360 4585 50  0000 L CNN
 F 1 "2.7kohm" V 2310 4580 50  0000 L CNN
-F 2 "Resistor_SMD:R_0402_1005Metric" H 2410 4760 50  0001 C CNN
+F 2 "Resistor_SMD:R_0603_1608Metric" H 2410 4760 50  0001 C CNN
 F 3 "" H 2410 4760 50  0001 C CNN
 	1    2410 4760
@@
 F 0 "C47" H 1685 4160 50  0000 L CNN
 F 1 "100nF" H 1685 4035 50  0000 L CNN
-F 2 "Capacitor_SMD:C_0402_1005Metric" H 1785 4085 50  0001 C CNN
+F 2 "Capacitor_SMD:C_0603_1608Metric" H 1785 4085 50  0001 C CNN
 F 3 "" H 1785 4085 50  0001 C CNN
 	1    1785 4085
@@
 F 0 "C51" V 3010 4385 50  0000 L CNN
 F 1 "10nF" V 3160 4235 50  0000 L CNN
-F 2 "Capacitor_SMD:C_0402_1005Metric" H 3060 4360 50  0001 C CNN
+F 2 "Capacitor_SMD:C_0603_1608Metric" H 3060 4360 50  0001 C CNN
 F 3 "" H 3060 4360 50  0001 C CNN
 	1    3060 4360
@@
 F 0 "C48" H 1795 4630 50  0000 L CNN
 F 1 "100nF" H 1795 4505 50  0000 L CNN
-F 2 "Capacitor_SMD:C_0402_1005Metric" H 1895 4555 50  0001 C CNN
+F 2 "Capacitor_SMD:C_0603_1608Metric" H 1895 4555 50  0001 C CNN
 F 3 "" H 1895 4555 50  0001 C CNN
 	1    1895 4555
@@
 F 0 "C62" H 7580 2380 50  0000 L CNN
 F 1 "0.8nF" V 7625 2070 50  0000 L CNN
-F 2 "Capacitor_SMD:C_0402_1005Metric" H 7570 2310 50  0001 C CNN
+F 2 "Capacitor_SMD:C_0603_1608Metric" H 7570 2310 50  0001 C CNN
 F 3 "" H 7570 2310 50  0001 C CNN
 	1    7570 2310
@@
 F 0 "C74" V 9690 2340 50  0000 L CNN
 F 1 "0.8nF" V 9615 2340 50  0000 L CNN
-F 2 "Capacitor_SMD:C_0402_1005Metric" H 9650 2315 50  0001 C CNN
+F 2 "Capacitor_SMD:C_0603_1608Metric" H 9650 2315 50  0001 C CNN
 F 3 "" H 9650 2315 50  0001 C CNN
 	1    9650 2315
@@
 F 0 "C65" V 7880 530 50  0000 L CNN
 F 1 "10nF" V 7875 740 50  0000 L CNN
-F 2 "Capacitor_SMD:C_0402_1005Metric" H 7915 705 50  0001 C CNN
+F 2 "Capacitor_SMD:C_0603_1608Metric" H 7915 705 50  0001 C CNN
 F 3 "" H 7915 705 50  0001 C CNN
 	1    7915 705
@@
 F 0 "C67" H 9110 4735 50  0000 L CNN
 F 1 "40nF" H 9000 4540 50  0000 L CNN
-F 2 "Capacitor_SMD:C_0402_1005Metric" H 9100 4665 50  0001 C CNN
+F 2 "Capacitor_SMD:C_0603_1608Metric" H 9100 4665 50  0001 C CNN
 F 3 "" H 9100 4665 50  0000 C CNN
 	1    9100 4665
@@
 F 0 "C69" H 9285 4735 50  0000 L CNN
 F 1 "40nF" H 9180 4600 50  0000 L CNN
-F 2 "Capacitor_SMD:C_0402_1005Metric" H 9275 4665 50  0001 C CNN
+F 2 "Capacitor_SMD:C_0603_1608Metric" H 9275 4665 50  0001 C CNN
 F 3 "" H 9275 4665 50  0000 C CNN
 	1    9275 4665
@@
 F 0 "C71" H 9485 4735 50  0000 L CNN
 F 1 "40nF" H 9380 4555 50  0000 L CNN
-F 2 "Capacitor_SMD:C_0402_1005Metric" H 9475 4665 50  0001 C CNN
+F 2 "Capacitor_SMD:C_0603_1608Metric" H 9475 4665 50  0001 C CNN
 F 3 "" H 9475 4665 50  0000 C CNN
 	1    9475 4665
@@
 F 0 "C75" H 9710 4735 50  0000 L CNN
 F 1 "40nF" H 9600 4595 50  0000 L CNN
-F 2 "Capacitor_SMD:C_0402_1005Metric" H 9700 4665 50  0001 C CNN
+F 2 "Capacitor_SMD:C_0603_1608Metric" H 9700 4665 50  0001 C CNN
 F 3 "" H 9700 4665 50  0000 C CNN
 	1    9700 4665
@@
 F 0 "C59" H 7480 3980 50  0000 L CNN
 F 1 "10nF" H 7480 3830 50  0000 L CNN
-F 2 "Capacitor_SMD:C_0402_1005Metric" H 7470 3910 50  0001 C CNN
+F 2 "Capacitor_SMD:C_0603_1608Metric" H 7470 3910 50  0001 C CNN
 F 3 "" H 7470 3910 50  0001 C CNN
 	1    7470 3910
@@
 F 0 "C50" H 1910 7345 50  0000 L CNN
 F 1 "10uF" H 1910 7195 50  0000 L CNN
-F 2 "Capacitor_SMD:C_0402_1005Metric" H 1900 7275 50  0001 C CNN
+F 2 "Capacitor_SMD:C_0603_1608Metric" H 1900 7275 50  0001 C CNN
 F 3 "" H 1900 7275 50  0000 C CNN
 	1    1900 7275
@@
 F 0 "C44" H 785 7345 50  0000 L CNN
 F 1 "100nF" H 785 7195 50  0000 L CNN
-F 2 "Capacitor_SMD:C_0402_1005Metric" H 775 7275 50  0001 C CNN
+F 2 "Capacitor_SMD:C_0603_1608Metric" H 775 7275 50  0001 C CNN
 F 3 "" H 775 7275 50  0000 C CNN
 	1    775  7275
