File: hardware/AD9954sheet.sch (KiCad schematic (older format))
At the start: 40 parts, among them IC2 AD9954

Commit message: Finished work on Receiver RPi shield. Changed CLK to SI5351A. Minimized footprints for almost all Tayloe detector ICs. Added -12V to audio opamps. Prepared board for coexisting with Hifiberry.
Parts:
- R14, R15, R17: footprint Resistor_SMD:R_0603_1608Metric -> Resistor_SMD:R_0805_2012Metric
Changed lines of the file:
@@
 EESchema Schematic File Version 4
 LIBS:rf-receiver-cache
-EELAYER 26 0
+EELAYER 29 0
 EELAYER END
 $Descr A4 11693 8268
 encoding utf-8
-Sheet 4 7
+Sheet 2 4
 Title ""
 Date ""
@@
 F 0 "R17" H 6580 3220 50  0000 L CNN
 F 1 "50ohm" H 6250 3200 50  0000 L CNN
-F 2 "Resistor_SMD:R_0603_1608Metric" H 6550 3200 50  0001 C CNN
+F 2 "Resistor_SMD:R_0805_2012Metric" H 6550 3200 50  0001 C CNN
 F 3 "" H 6550 3200 50  0000 C CNN
 	1    6550 3200
@@
 F 0 "R14" V 3925 4825 50  0000 L CNN
 F 1 "50ohm" V 3975 4700 50  0000 L CNN
-F 2 "Resistor_SMD:R_0603_1608Metric" H 4050 4850 50  0001 C CNN
+F 2 "Resistor_SMD:R_0805_2012Metric" H 4050 4850 50  0001 C CNN
 F 3 "" H 4050 4850 50  0000 C CNN
 	1    4050 4850
@@
 F 0 "R15" V 4125 4925 50  0000 L CNN
 F 1 "50ohm" V 3975 4850 50  0000 L CNN
-F 2 "Resistor_SMD:R_0603_1608Metric" H 4050 5000 50  0001 C CNN
+F 2 "Resistor_SMD:R_0805_2012Metric" H 4050 5000 50  0001 C CNN
 F 3 "" H 4050 5000 50  0000 C CNN
 	1    4050 5000

Commit message: Added rpi changes - seems weird that I forgot that for so long
Connections:
- net OSK is gone; now on net GND: IC2.46 (OSK)
Changed lines of the file:
@@
 Text HLabel 3450 1900 1    60   Input ~ 0
 PS0
-Text HLabel 3600 1900 1    60   Input ~ 0
-OSK
 Text HLabel 3750 1900 1    60   Output ~ 0
 SYNC_CLK
@@
 Wire Wire Line
 	3675 7050 3800 7050
+Text Label 3600 1475 3    60   ~ 0
+DGND
+Wire Wire Line
+	3600 1900 3600 1475
 $EndSCHEMATC
