File: hardware/powersheet.sch (KiCad schematic (older format))
At the start: 17 parts, among them U10 TPS62173DSG, U11 MIC5504-1.8YM5, U12 MIC5504-1.8YM5

Commit message: Finished work on Receiver RPi shield. Changed CLK to SI5351A. Minimized footprints for almost all Tayloe detector ICs. Added -12V to audio opamps. Prepared board for coexisting with Hifiberry.
Parts:
- removed C76: 100uF, Capacitor_SMD:CP_Elec_6.3x7.7, symbol Device:CP_Small
- removed C77, C79: 100nF, Capacitor_SMD:C_0603_1608Metric, symbol Device:C_Small
- removed C78: 22uF, Capacitor_SMD:C_0603_1608Metric, symbol Device:C_Small
- removed C?: CP_Small, symbol Device:CP_Small
- removed FL1: ACP3225, athir:ACP3225, symbol athir:ACP3225
- removed L8: 2.2uH, athir:XFL3012, symbol Device:L_Small
- removed PSU+1: PSU+, TestPoint:TestPoint_THTPad_2.0x2.0mm_Drill1.0mm, symbol Connector:TestPoint
- removed PSU-1: PSU-, TestPoint:TestPoint_THTPad_2.0x2.0mm_Drill1.0mm, symbol Connector:TestPoint
- removed R33: 100k, Resistor_SMD:R_0603_1608Metric, symbol Device:R_Small
- removed U10: TPS62173DSG, Package_SON:WSON-8-1EP_2x2mm_P0.5mm_EP0.9x1.6mm_ThermalVias, symbol athir:TPS62173DSG
- added C10: 10uF, Capacitor_SMD:C_0603_1608Metric, symbol Device:CP_Small
- added C11, C8: 47uF/100uF, Capacitor_SMD:CP_Elec_6.3x7.7, symbol Device:CP_Small
- added C12, C13: 100nF, Capacitor_SMD:C_0603_1608Metric, symbol Device:C_Small
- added C55, C58: 10u, Capacitor_SMD:C_0603_1608Metric, symbol Device:CP_Small
- added C60: 100n, Capacitor_SMD:C_0603_1608Metric, symbol Device:CP_Small
- added C7, C9: 22uF, Capacitor_SMD:CP_Elec_6.3x7.7, symbol Device:CP_Small
- added C81: 10p, Capacitor_SMD:C_0603_1608Metric, symbol Device:CP_Small
- added FL1: ACM90V-701-2PL-TL00, symbol Device:EMI_Filter_LL_1423
- added J4: Jack-DC, symbol Connector:Jack-DC
- added L1: 3.3uH, athir:XFL3012, symbol Device:L_Small
- added R3: 10k 1%, Resistor_SMD:R_0603_1608Metric, symbol Device:R_Small
- added R4: 10k, Resistor_SMD:R_0603_1608Metric, symbol Device:R_Small
- added R5: 54k9 1%, Resistor_SMD:R_0603_1608Metric, symbol Device:R_Small
- added U2: TPS565208, Package_TO_SOT_SMD:SOT-23-6, symbol athir:TPS565208
- added U6: LMC7660, Package_SO:SOIC-8_3.9x4.9mm_P1.27mm, symbol Regulator_SwitchedCapacitor:LMC7660
Connections:
- net labels added: -12V
- wire segments 82 -> 114
- no-connect marks 0 -> 1
Other:
- note added: "ERSTAT MED: \nLM2677SX-5.0/NOPB\n5V @ 5A\n-> RPI support"

Commit message: Added rpi changes - seems weird that I forgot that for so long
Parts:
- removed C10: 10uF, Capacitor_SMD:C_0603_1608Metric, symbol Device:CP_Small
- removed C11: 47uF/100uF, Capacitor_SMD:CP_Elec_6.3x7.7, symbol Device:CP_Small
- removed C55, C58: 10u, Capacitor_SMD:C_0603_1608Metric, symbol Device:CP_Small
- removed C60: 100n, Capacitor_SMD:C_0603_1608Metric, symbol Device:CP_Small
- removed C7, C9: 22uF, Capacitor_SMD:CP_Elec_6.3x7.7, symbol Device:CP_Small
- removed C80, C82: 100nF, Capacitor_SMD:C_0603_1608Metric, symbol Device:C_Small
- removed C81: 10p, Capacitor_SMD:C_0603_1608Metric, symbol Device:CP_Small
- removed C83, C85: 10uF, Capacitor_SMD:C_0603_1608Metric, symbol Device:C_Small
- removed J4: Jack-DC, symbol Connector:Jack-DC
- removed R3: 10k 1%, Resistor_SMD:R_0603_1608Metric, symbol Device:R_Small
- removed R4: 10k, Resistor_SMD:R_0603_1608Metric, symbol Device:R_Small
- removed R5: 54k9 1%, Resistor_SMD:R_0603_1608Metric, symbol Device:R_Small
- removed U11, U12: MIC5504-1.8YM5, Package_TO_SOT_SMD:SOT-23-5, symbol Regulator_Linear:MIC5504-1.8YM5
- removed U2: TPS565208, Package_TO_SOT_SMD:SOT-23-6, symbol athir:TPS565208
- removed U6: LMC7660, Package_SO:SOIC-8_3.9x4.9mm_P1.27mm, symbol Regulator_SwitchedCapacitor:LMC7660
- added C10, C11, C9: 22uF, Capacitor_SMD:C_0805_2012Metric, symbol Device:C_Small
- added C22: 100nF, Capacitor_SMD:C_0603_1608Metric, symbol Device:C_Small
- added D3: D_Small_ALT, Diode_SMD:D_SOD-323_HandSoldering, symbol Device:D_Small_ALT
- added FL2, FL3: ACP3225, athir:ACP3225, symbol athir:ACP3225
- added J10: 12P_VIN, athir:FASTON63951-1, symbol Connector:Conn_01x01_Male
- added J12: 12N_VIN, athir:FASTON63951-1, symbol Connector:Conn_01x01_Male
- added J4: 5_VIN, athir:FASTON63951-1, symbol Connector:Conn_01x01_Male
- added J9: GND_IN, athir:FASTON63951-1, symbol Connector:Conn_01x01_Male
- added TP10: 5V_TP, athir:testpoint_probe, symbol Connector:TestPoint
- added TP11: 12V_TP, athir:testpoint_probe, symbol Connector:TestPoint
- added TP12: -12V_TP, athir:testpoint_probe, symbol Connector:TestPoint
- added TP14: 3.3VA, athir:testpoint_probe, symbol Connector:TestPoint
- added TP15: 3.3V, athir:testpoint_probe, symbol Connector:TestPoint
- added TP9: GND, athir:testpoint_probe, symbol Connector:TestPoint
- C8: footprint Capacitor_SMD:CP_Elec_6.3x7.7 -> Capacitor_SMD:CP_Elec_6.3x5.4
- FL1: footprint (none) -> athir:ACM70V-701-2PL-TL00
- L1: value 3.3uH -> 47+uH; footprint athir:XFL3012 -> Inductor_SMD:L_Wuerth_HCM-7050
Connections:
- net labels added: +3.3V, +3.3VA
- net labels removed: +1V8, VAA
- wire segments 114 -> 71
- no-connect marks 1 -> 0
Other:
- note added: "ERSTAT MED:\nICL7660S\nfor -12V support"
- note removed: "ERSTAT MED: \nLM2677SX-5.0/NOPB\n5V @ 5A\n-> RPI support"
- moved on the sheet: FL1

Commit message: Sorry future me
Parts:
- added C33: 47uF/100uF, Capacitor_SMD:CP_Elec_6.3x5.4, symbol Device:CP_Small
- added D4: D_Small_ALT, athir:SOD128, symbol Device:D_Small_ALT
- added TP18: GND, athir:testpoint_probe, symbol Connector:TestPoint
Connections:
- net +5V: now also C33.1
- net GND: now also C33.2, TP18.1
- net at D3.1 (K), FL1.2: now also D4.1 (K)
- net at D3.2 (A), J4.1 (Pin_1): now also D4.2 (A)
Changed lines of the file:
@@
 $Descr A4 11693 8268
 encoding utf-8
-Sheet 3 3
+Sheet 4 4
 Title ""
 Date ""
@@
 	3445 4495 3445 4440
 Wire Wire Line
-	3150 4495 3445 4495
+	3150 4495 3300 4495
 Wire Wire Line
 	1705 4755 1705 4750
@@
 $EndComp
 Wire Wire Line
-	1665 4550 1705 4550
+	1665 4550 1690 4550
 Wire Wire Line
 	1390 4500 1390 4550
 Wire Wire Line
-	1390 4550 1465 4550
+	1390 4550 1430 4550
+$Comp
+L Connector:TestPoint TP?
+U 1 1 5E5CA4EA
+P 4205 4025
+AR Path="/5C4FD13D/5E5CA4EA" Ref="TP?"  Part="1"
+AR Path="/5C517D7D/5E5CA4EA" Ref="TP18"  Part="1"
+F 0 "TP18" H 4263 4145 50  0000 L CNN
+F 1 "GND" H 4263 4054 50  0000 L CNN
+F 2 "athir:testpoint_probe" H 4405 4025 50  0001 C CNN
+F 3 "~" H 4405 4025 50  0001 C CNN
+	1    4205 4025
+	1    0    0    -1
+$EndComp
+$Comp
+L power:GND #PWR?
+U 1 1 5E5CA4F4
+P 4205 4065
+AR Path="/5C4FD13D/5E5CA4F4" Ref="#PWR?"  Part="1"
+AR Path="/5C517D7D/5E5CA4F4" Ref="#PWR011"  Part="1"
+F 0 "#PWR011" H 4205 3815 50  0001 C CNN
+F 1 "GND" H 4210 3892 50  0000 C CNN
+F 2 "" H 4205 4065 50  0001 C CNN
+F 3 "" H 4205 4065 50  0001 C CNN
+	1    4205 4065
+	1    0    0    -1
+$EndComp
+Wire Wire Line
+	4205 4025 4205 4065
+$Comp
+L Device:D_Small_ALT D4
+U 1 1 5E614377
+P 1560 4400
+F 0 "D4" H 1560 4195 50  0000 C CNN
+F 1 "D_Small_ALT" H 1560 4286 50  0000 C CNN
+F 2 "athir:SOD128" V 1560 4400 50  0001 C CNN
+F 3 "~" V 1560 4400 50  0001 C CNN
+	1    1560 4400
+	-1   0    0    1
+$EndComp
+Wire Wire Line
+	1690 4400 1690 4550
+Connection ~ 1690 4550
+Wire Wire Line
+	1690 4550 1705 4550
+Wire Wire Line
+	1460 4400 1430 4400
+Wire Wire Line
+	1430 4400 1430 4550
+Connection ~ 1430 4550
+Wire Wire Line
+	1430 4550 1465 4550
+Wire Wire Line
+	1660 4400 1690 4400
+$Comp
+L Device:CP_Small C33
+U 1 1 5E7102DA
+P 3300 4650
+F 0 "C33" H 3400 4725 50  0000 R CNN
+F 1 "47uF/100uF" H 3675 4575 50  0000 R CNN
+F 2 "Capacitor_SMD:CP_Elec_6.3x5.4" H 3300 4650 50  0001 C CNN
+F 3 "~" H 3300 4650 50  0001 C CNN
+	1    3300 4650
+	1    0    0    -1
+$EndComp
+Wire Wire Line
+	3300 4550 3300 4495
+Connection ~ 3300 4495
+Wire Wire Line
+	3300 4495 3445 4495
+Wire Wire Line
+	3300 4750 3300 4795
+Wire Wire Line
+	3300 4795 3185 4795
+Connection ~ 3185 4795
 $EndSCHEMATC
