File: hardware/tayloesheet.sch (KiCad schematic (older format))
At the start: 53 parts, among them IC3 74LVC74, J1 Conn_01x05_Female, J2 Conn_Coaxial, U4 MIC5504-3.3YM5, U5 OPA300, U7 Transformer, U8 NE5532, U9 74CBTLV3253

Commit message: Finished work on Receiver RPi shield. Changed CLK to SI5351A. Minimized footprints for almost all Tayloe detector ICs. Added -12V to audio opamps. Prepared board for coexisting with Hifiberry.
Parts:
- removed J1: Conn_01x05_Female, athir:SJ1-35235, symbol Connector:Conn_01x05_Female
- added C5: 10uF, Capacitor_SMD:C_0603_1608Metric, symbol Device:C_Small
- added C6: 10nF, Capacitor_SMD:C_0603_1608Metric, symbol Device:C_Small
- IC3: value 74LVC74 -> 74LVC74ABQ; footprint Package_SO:SOIC-14_3.9x8.7mm_P1.27mm -> Package_DFN_QFN:DFN-12-1EP_3x4mm_P0.5mm_EP1.7x3.3mm
- R21: footprint Resistor_SMD:R_0603_1608Metric -> Resistor_SMD:R_0805_2012Metric
Connections:
- net GND: now also C5.1, C6.1; no longer U8.4 (V-)
- new net -12V: C5.2, C6.2, U8.4 (V-)
- no-connect marks 1 -> 0
Other:
- note added: "OPA2211AIDRGT\nWSON-8\n1.1nV\nmindre footprint\n9,95 €"
Changed lines of the file:
@@
 EESchema Schematic File Version 4
 LIBS:rf-receiver-cache
-EELAYER 26 0
+EELAYER 29 0
 EELAYER END
 $Descr A4 11693 8268
 encoding utf-8
-Sheet 6 7
+Sheet 3 4
 Title "Tayloe Detector"
 Date "2017-03-29"
@@
 P 3165 3440
 F 0 "IC3" H 3965 3690 60  0000 C CNN
-F 1 "74LVC74" H 3765 4490 60  0000 C CNN
-F 2 "Package_SO:SOIC-14_3.9x8.7mm_P1.27mm" H 3765 3990 60  0001 C CNN
+F 1 "74LVC74ABQ" H 3765 4490 60  0000 C CNN
+F 2 "Package_DFN_QFN:DFN-12-1EP_3x4mm_P0.5mm_EP1.7x3.3mm" H 3765 3990 60  0001 C CNN
 F 3 "" H 3765 3990 60  0000 C CNN
 	1    3165 3440
@@
 Text Label 7080 4360 2    60   ~ 0
 LO_IN_B
-$Comp
-L power:GND #PWR085
-U 1 1 58E53A66
-P 7575 1475
-F 0 "#PWR085" H 7575 1225 50  0001 C CNN
-F 1 "GND" H 7575 1325 50  0000 C CNN
-F 2 "" H 7575 1475 50  0001 C CNN
-F 3 "" H 7575 1475 50  0001 C CNN
-	1    7575 1475
-	1    0    0    -1
-$EndComp
 $Comp
 L Amplifier_Operational:NE5532 U8
@@
 F 0 "R21" V 1360 4410 50  0000 L CNN
 F 1 "50ohm" V 1510 4310 50  0000 L CNN
-F 2 "Resistor_SMD:R_0603_1608Metric" H 1435 4460 50  0001 C CNN
+F 2 "Resistor_SMD:R_0805_2012Metric" H 1435 4460 50  0001 C CNN
 F 3 "" H 1435 4460 50  0001 C CNN
 	1    1435 4460
@@
 	1    0    0    -1
 $EndComp
-$Comp
-L power:GND #PWR080
-U 1 1 5A247566
-P 4425 1600
-F 0 "#PWR080" H 4425 1350 50  0001 C CNN
-F 1 "GND" H 4430 1427 50  0000 C CNN
-F 2 "" H 4425 1600 50  0001 C CNN
-F 3 "" H 4425 1600 50  0001 C CNN
-	1    4425 1600
-	1    0    0    -1
-$EndComp
-Text Label 4250 1475 0    60   ~ 0
-Q_OUT
-Text Label 4250 1375 0    60   ~ 0
-I_OUT
 $Comp
 L power:PWR_FLAG #FLG07
@@
 	1900 6925 1900 7050
 $Comp
-L Connector:Conn_01x05_Female J1
-U 1 1 5C4A7415
-P 4050 1375
-F 0 "J1" H 3944 950 50  0000 C CNN
-F 1 "Conn_01x05_Female" H 3944 1041 50  0000 C CNN
-F 2 "athir:SJ1-35235" H 4050 1375 50  0001 C CNN
-F 3 "~" H 4050 1375 50  0001 C CNN
-	1    4050 1375
+L power:-12V #PWR0118
+U 1 1 5D91C97B
+P 7575 1475
+F 0 "#PWR0118" H 7575 1575 50  0001 C CNN
+F 1 "-12V" H 7590 1648 50  0000 C CNN
+F 2 "" H 7575 1475 50  0001 C CNN
+F 3 "" H 7575 1475 50  0001 C CNN
+	1    7575 1475
 	-1   0    0    1
 $EndComp
-Wire Wire Line
-	4425 1600 4425 1575
-Wire Wire Line
-	4425 1575 4250 1575
-NoConn ~ 4250 1175
-Wire Wire Line
-	4250 1275 4425 1275
-Wire Wire Line
-	4425 1275 4425 1575
-Connection ~ 4425 1575
+$Comp
+L Device:C_Small C5
+U 1 1 5D91DF94
+P 8200 1500
+F 0 "C5" V 8240 1525 50  0000 L CNN
+F 1 "10uF" V 8250 1280 50  0000 L CNN
+F 2 "Capacitor_SMD:C_0603_1608Metric" H 8200 1500 50  0001 C CNN
+F 3 "" H 8200 1500 50  0001 C CNN
+	1    8200 1500
+	-1   0    0    1
+$EndComp
+$Comp
+L Device:C_Small C6
+U 1 1 5D91EE50
+P 8350 1500
+F 0 "C6" V 8315 1325 50  0000 L CNN
+F 1 "10nF" V 8310 1535 50  0000 L CNN
+F 2 "Capacitor_SMD:C_0603_1608Metric" H 8350 1500 50  0001 C CNN
+F 3 "" H 8350 1500 50  0001 C CNN
+	1    8350 1500
+	-1   0    0    1
+$EndComp
+Wire Wire Line
+	8000 1475 8000 1350
+Wire Wire Line
+	8000 1350 8200 1350
+Wire Wire Line
+	8350 1350 8350 1400
+Wire Wire Line
+	7575 1475 8000 1475
+Connection ~ 7575 1475
+Wire Wire Line
+	8200 1400 8200 1350
+Connection ~ 8200 1350
+Wire Wire Line
+	8200 1350 8350 1350
+$Comp
+L power:GND #PWR0119
+U 1 1 5D94C222
+P 8250 1650
+F 0 "#PWR0119" H 8250 1400 50  0001 C CNN
+F 1 "GND" H 8255 1477 50  0000 C CNN
+F 2 "" H 8250 1650 50  0001 C CNN
+F 3 "" H 8250 1650 50  0001 C CNN
+	1    8250 1650
+	1    0    0    -1
+$EndComp
+Wire Wire Line
+	8250 1650 8250 1625
+Wire Wire Line
+	8250 1625 8200 1625
+Wire Wire Line
+	8200 1625 8200 1600
+Wire Wire Line
+	8350 1600 8350 1625
+Wire Wire Line
+	8350 1625 8250 1625
+Connection ~ 8250 1625
+Text Notes 9300 2850 0    50   ~ 0
+OPA2211AIDRGT\nWSON-8\n1.1nV\nmindre footprint\n9,95 €
 $EndSCHEMATC

Commit message: Added rpi changes - seems weird that I forgot that for so long
Parts:
- removed R30, R32: 10kohm, Resistor_SMD:R_0603_1608Metric, symbol Device:R_Small
- added C21: 100nF, Capacitor_SMD:C_0603_1608Metric, symbol Device:C_Small
- added J5, J7: RF_Shield_One_Piece, RF_Shielding:Laird_Technologies_BMI-S-102_16.50x16.50mm, symbol Device:RF_Shield_One_Piece
- added J6: RF_Shield_One_Piece, RF_Shielding:Laird_Technologies_BMI-S-101_13.66x12.70mm, symbol Device:RF_Shield_One_Piece
- added TP1: RF_DC_BIAS, athir:testpoint_probe, symbol Connector:TestPoint
- C44: value 100nF -> 10uF
- C52: value 47uF -> 22uF; footprint Capacitor_SMD:CP_Elec_6.3x7.7 -> Capacitor_SMD:C_0805_2012Metric
- C56: footprint Capacitor_SMD:C_0603_1608Metric -> Capacitor_SMD:CP_Elec_4x5.4
- IC3: footprint Package_DFN_QFN:DFN-12-1EP_3x4mm_P0.5mm_EP1.7x3.3mm -> athir:DHVQFN14
- TP3, TP4, TP5, TP6, TP7, TP8: footprint TestPoint:TestPoint_Pad_D1.0mm -> athir:testpoint_probe
- U8: value NE5532 -> OPA167B-DRG; footprint Package_SO:SOIC-8_3.9x4.9mm_P1.27mm -> Package_SON:SON-8-1EP_3x2mm_P0.5mm_EP1.4x1.6mm
- U9: footprint Package_SO:TSSOP-16_4.4x5mm_P0.65mm -> athir:PVQFN16
Connections:
- net +3V3: now also C21.1
- net DC_BIAS: now also TP1.1
- net GND: now also C21.2, J5.1 (Shield), J6.1 (Shield), J7.1 (Shield)
Other:
- note added: "OPA1678 DRG - SON-8\nPin compatible.\nhttp://www.ti.com/lit/ds/symlink/opa1678.pdf"

Commit message: HW: Fixed SMA footprint and 74x3253 footprint
Parts:
- J2: footprint Connector_Coaxial:SMA_Amphenol_132289_EdgeMount -> athir:SMA_Edge-mount
Changed lines of the file:
@@
 F 0 "J2" H 2049 651 50  0000 L CNN
 F 1 "Conn_Coaxial" H 2049 560 50  0000 L CNN
-F 2 "Connector_Coaxial:SMA_Amphenol_132289_EdgeMount" H 1950 675 50  0001 C CNN
+F 2 "athir:SMA_Edge-mount" H 1950 675 50  0001 C CNN
 F 3 "" H 1950 675 50  0001 C CNN
 	1    1950 675

Commit message: Sorry future me
Parts:
- added R10: 50ohm, Resistor_SMD:R_0603_1608Metric, symbol Device:R_Small
- C53, C63: value 0.1uF -> 100nF
- J2: value Conn_Coaxial -> ANT
- U6: renamed from IC3; footprint athir:DHVQFN14 -> athir:74LVC74ABQ; symbol athir:74LVC74 -> athir:74LVC74ABQ
Connections:
- net GND: now also R10.2
- net LO_IN: now also R10.1
- net RF_IN_A: no longer J2.1 (In)
- new net 30 MHz Low Pass Filter/IN: J2.1 (In)
Other:
- moved on the sheet: J2
Changed lines of the file:
@@
 $Descr A4 11693 8268
 encoding utf-8
-Sheet 2 3
+Sheet 2 4
 Title "Tayloe Detector"
 Date "2017-03-29"
@@
 $EndComp
 $Comp
-L athir:74LVC74 IC3
+L athir:74LVC74ABQ U6
 U 1 1 58946947
 P 3165 3440
-F 0 "IC3" H 3965 3690 60  0000 C CNN
+F 0 "U6" H 3965 3690 60  0000 C CNN
 F 1 "74LVC74ABQ" H 3765 4490 60  0000 C CNN
-F 2 "athir:DHVQFN14" H 3765 3990 60  0001 C CNN
+F 2 "athir:74LVC74ABQ" H 3765 3990 60  0001 C CNN
 F 3 "" H 3765 3990 60  0000 C CNN
 	1    3165 3440
@@
 P 4465 2490
 F 0 "C53" H 4515 2540 50  0000 L CNN
-F 1 "0.1uF" H 4475 2410 50  0000 L CNN
+F 1 "100nF" H 4475 2410 50  0000 L CNN
 F 2 "Capacitor_SMD:C_0603_1608Metric" H 4465 2490 50  0001 C CNN
 F 3 "" H 4465 2490 50  0000 C CNN
@@
 P 7635 3910
 F 0 "C63" H 7645 3980 50  0000 L CNN
-F 1 "0.1uF" H 7645 3830 50  0000 L CNN
+F 1 "100nF" H 7645 3830 50  0000 L CNN
 F 2 "Capacitor_SMD:C_0603_1608Metric" H 7635 3910 50  0001 C CNN
 F 3 "" H 7635 3910 50  0000 C CNN
@@
 L power:GND #PWR062
 U 1 1 58DD6ED5
-P 1950 900
-F 0 "#PWR062" H 1950 650 50  0001 C CNN
-F 1 "GND" H 1950 750 50  0000 C CNN
-F 2 "" H 1950 900 50  0001 C CNN
-F 3 "" H 1950 900 50  0001 C CNN
-	1    1950 900
-	1    0    0    -1
-$EndComp
-Text Label 1750 675  2    60   ~ 0
+P 2580 1025
+F 0 "#PWR062" H 2580 775 50  0001 C CNN
+F 1 "GND" H 2580 875 50  0000 C CNN
+F 2 "" H 2580 1025 50  0001 C CNN
+F 3 "" H 2580 1025 50  0001 C CNN
+	1    2580 1025
+	1    0    0    -1
+$EndComp
+Text Label 4080 775  0    60   ~ 0
 RF_IN_A
 Text Label 5310 4665 2    60   ~ 0
@@
 L Connector:Conn_Coaxial J2
 U 1 1 5A1CD076
-P 1950 675
-F 0 "J2" H 2049 651 50  0000 L CNN
-F 1 "Conn_Coaxial" H 2049 560 50  0000 L CNN
-F 2 "athir:SMA_Edge-mount" H 1950 675 50  0001 C CNN
-F 3 "" H 1950 675 50  0001 C CNN
-	1    1950 675
-	1    0    0    -1
+P 2580 800
+F 0 "J2" H 2679 776 50  0000 L CNN
+F 1 "ANT" H 2679 685 50  0000 L CNN
+F 2 "athir:SMA_Edge-mount" H 2580 800 50  0001 C CNN
+F 3 "" H 2580 800 50  0001 C CNN
+	1    2580 800
+	-1   0    0    -1
 $EndComp
 $Comp
@@
 Connection ~ 3315 2490
 Wire Notes Line
-	5415 3390 565  3390
+	5415 3405 565  3405
 Wire Notes Line
 	565  3390 565  2040
@@
 	3350 3090 3350 3110
 Wire Wire Line
-	1950 900  1950 875
+	2580 1025 2580 1000
 Wire Wire Line
 	1855 4225 1855 4855
@@
 LO_IN
 Wire Wire Line
-	2690 2890 3180 2890
+	2690 2890 2830 2890
 $Comp
 L Regulator_Linear:MIC5504-3.3YM5 U?
@@
 Wire Wire Line
 	5975 3885 6010 3885
+$Sheet
+S 2885 715  1195 270
+U 5E5AECBB
+F0 "30 MHz Low Pass Filter" 50
+F1 "30mhzlp.sch" 50
+F2 "IN" I L 2885 800 50
+F3 "OUT" O R 4080 775 50
+$EndSheet
+Wire Wire Line
+	2885 800  2780 800
+$Comp
+L Device:R_Small R10
+U 1 1 5E760658
+P 2830 3060
+F 0 "R10" V 2690 3020 50  0000 L CNN
+F 1 "50ohm" V 2905 2910 50  0000 L CNN
+F 2 "Resistor_SMD:R_0603_1608Metric" H 2830 3060 50  0001 C CNN
+F 3 "" H 2830 3060 50  0001 C CNN
+	1    2830 3060
+	1    0    0    -1
+$EndComp
+Wire Wire Line
+	2830 2960 2830 2890
+Connection ~ 2830 2890
+Wire Wire Line
+	2830 2890 3180 2890
+$Comp
+L power:GND #PWR0133
+U 1 1 5E77901C
+P 2830 3205
+F 0 "#PWR0133" H 2830 2955 50  0001 C CNN
+F 1 "GND" H 2830 3055 50  0000 C CNN
+F 2 "" H 2830 3205 50  0000 C CNN
+F 3 "" H 2830 3205 50  0000 C CNN
+	1    2830 3205
+	1    0    0    -1
+$EndComp
+Wire Wire Line
+	2830 3205 2830 3160
 $EndSCHEMATC
