File: hardware/30mhzLP/30mhzLP.kicad_pcb (KiCad board)
At the start: 2 copper layers, 58 x 35.5 mm, 9 parts, among them J1 Conn_Coaxial, J2 Conn_Coaxial

Commit message: temp
Parts:
- removed L4: 300nH, athir:2222SQ-301
- added C4: 220p, Capacitor_SMD:C_0603_1608Metric, F.Cu at (140.8, 112.8)
- added C5: 270p, Capacitor_SMD:C_0603_1608Metric, F.Cu at (144.2, 113.5)
- added C6: 130p, Capacitor_SMD:C_0603_1608Metric, F.Cu at (147.5, 112.8)
- added C7: 270p, Capacitor_SMD:C_0603_1608Metric, F.Cu at (151.0, 113.5)
- added R1: 50, Resistor_SMD:R_0805_2012Metric, F.Cu at (128.5, 110.0)
- C1, C3: value 150pF -> 330p
- C2: value 180pF -> 39p
- L1: value 300nH -> 180n; footprint athir:2222SQ-301 -> Inductor_SMD:L_0805_2012Metric
- L2: value 560nH -> 100n; footprint Inductor_SMD:L_0603_1608Metric -> Inductor_SMD:L_0805_2012Metric
- L3: value 560nH -> 120n; footprint Inductor_SMD:L_0603_1608Metric -> Inductor_SMD:L_0805_2012Metric
- moved C3 13.8 mm to (137.2, 113.5), turned to 270 degrees
- moved J2 13.3 mm to (158.2, 112.2)
- moved C2 11.5 mm to (133.5, 112.8), turned to 180 degrees
- moved C1 9.75 mm to (128.5, 113.5), turned to 270 degrees
- moved L2 3.05 mm to (140.8, 110.5), turned to 0 degrees
- moved L1 3.01 mm to (133.5, 110.5), turned to 0 degrees
- moved L3 2.80 mm to (147.5, 110.5), turned to 0 degrees
- moved J1 0.25 mm to (118.8, 112.5)
Connections:
- C2 pad 2: GND -> Net-(C1-Pad1)
- C3 pad 1: Net-(C3-Pad1) -> Net-(C2-Pad1)
- J1 pad 1: Net-(J1-Pad1) -> Net-(C1-Pad1)
- J2 pad 1: Net-(J2-Pad1) -> Net-(C6-Pad1)
- L1 pad 1: Net-(J1-Pad1) -> Net-(C1-Pad1)
- L1 pad 2: Net-(C1-Pad1) -> Net-(C2-Pad1)
- L2 pad 1: Net-(C1-Pad1) -> Net-(C2-Pad1)
- L2 pad 2: Net-(C2-Pad1) -> Net-(C4-Pad1)
- L3 pad 1: Net-(C2-Pad1) -> Net-(C4-Pad1)
- L3 pad 2: Net-(C3-Pad1) -> Net-(C6-Pad1)
Routing:
- net Net-(J2-Pad1): track 21.3 -> 0.00 mm
- net Net-(J1-Pad1): track 14.6 -> 0.00 mm
- net Net-(C6-Pad1): track 0.00 -> 12.2 mm
- net Net-(C3-Pad1): track 12.0 -> 0.00 mm
- net Net-(C4-Pad1): track 0.00 -> 9.86 mm
- net Net-(C1-Pad1): track 14.0 -> 18.4 mm
- net Net-(C2-Pad1): track 6.02 -> 10.3 mm
- net GND: vias 65 -> 50
Other:
- board size 58 x 35.5 mm -> 45 x 35.5 mm
- board text added: "7th order 30MHz Lowpass Elliptic Ripple -3dB Stopband -60dB"
- board text added: "ATHIR - 1950 Rev. 2"
- board text removed: "30MHz Low-Pass 7th order Chebyshev ATHIR - 1919"
- board text removed: "Z0: 50 Ohm 40MHz: -27dB 50MHz: -44dB 60MHz: -58dB 70MHz: -68dB 80MHz: -77dB"
