File: hardware/30mhzLP/30mhzLP.sch (KiCad schematic (older format))
At the start: 10 parts, among them J1 Conn_Coaxial, J2 Conn_Coaxial

Commit message: temp
Parts:
- removed L4: 300nH, athir:2222SQ-301, symbol Device:L_Small
- added C4: 220p, Capacitor_SMD:C_0603_1608Metric, symbol Device:C_Small
- added C5, C7: 270p, Capacitor_SMD:C_0603_1608Metric, symbol Device:C_Small
- added C6: 130p, Capacitor_SMD:C_0603_1608Metric, symbol Device:C_Small
- C1, C3: value 150pF -> 330p
- C2: value 180pF -> 39p
- L1: value 300nH -> 180n; footprint athir:2222SQ-301 -> Inductor_SMD:L_0805_2012Metric
- L2: value 560nH -> 100n; footprint Inductor_SMD:L_0603_1608Metric -> Inductor_SMD:L_0805_2012Metric
- L3: value 560nH -> 120n; footprint Inductor_SMD:L_0603_1608Metric -> Inductor_SMD:L_0805_2012Metric
- R1: footprint (none) -> Resistor_SMD:R_0805_2012Metric
Connections:
- net GND: now also C5.2, C7.2; no longer C2.2
- net at L1.2, L2.1: now also C2.1, C3.1, C4.2; no longer C1.1
- net at J2.1 (In): now also L3.2, C6.1, C7.1
- net at J1.1 (In), L1.1, R1.1: now also C1.1, C2.2
- net at L2.2, L3.1: now also C4.1, C5.1, C6.2; no longer C2.1
